File: schematic/signalmesh.kicad_sch (KiCad schematic)
At the start: 23 parts, among them J1 FPGA I/O, J2 FPGA I/O, J8 FPGA I/O, J9 FPGA I/O, U1 NUCLEO-H753ZI, U2 NUCLEO-H753ZI, U3 NUCLEO-F303RE, U4 YAAJ_BluePill_Part_Like, U5 24LC256-I_SN, U6 BME280, U7 INA219AxD, U8 24LC256-I_SN, U9 NUCLEO-F446RE

Commit message: update schematic and pcb. errors
Parts:
- added C1, C2, C3, C4, C5: 0.1uf, Capacitor_SMD:C_0201_0603Metric, symbol Device:C_Small
- added J10, J11, J5, J6, J7: INA219_CONFIG, Connector_PinHeader_1.00mm:PinHeader_1x02_P1.00mm_Horizontal, symbol Connector_Generic:Conn_01x02
- added J12: AAM_DBG, Connector_PinHeader_1.00mm:PinHeader_1x03_P1.00mm_Horizontal, symbol Connector_Generic:Conn_01x03
- added J13: DSM_DBG, Connector_PinHeader_1.00mm:PinHeader_1x03_P1.00mm_Horizontal, symbol Connector_Generic:Conn_01x03
- added J4: TDM_DBG, Connector_PinHeader_1.00mm:PinHeader_1x03_P1.00mm_Horizontal, symbol Connector_Generic:Conn_01x03
- added R13, R14, R19, R20, R21, R22, R23, R24, R25, R26, R28: 10k, Resistor_SMD:R_0805_2012Metric_Pad1.20x1.40mm_HandSolder, symbol Device:R
- added TH1: 10k, OptoDevice:R_LDR_4.9x4.2mm_P2.54mm_Vertical, symbol Device:Thermistor
- added U10, U11, U12, U13: INA219AxD, Package_SO:SOIC-8_3.9x4.9mm_P1.27mm, symbol Sensor_Energy:INA219AxD
Connections:
- net 5V_TDM: now also C1.2, C2.2, C3.2, C4.2, C5.2, U10.5 (VS), U10.8 (IN+), U11.5 (VS), U11.8 (IN+), U12.5 (VS), U12.8 (IN+), U13.5 (VS), U13.8 (IN+)
- net GND: now also C1.1, C2.1, C3.1, C4.1, C5.1, J12.3 (Pin_3), J13.3 (Pin_3), J4.3 (Pin_3), R13.1, R14.1, R20.1, R21.1, R22.1, R23.1, R24.1, R25.1, R26.1, R28.1, TH1.1, U10.6 (GND), U11.6 (GND), U12.6 (GND), U13.6 (GND); no longer U8.2 (A1)
- net I2C1_SCL_TDM: now also U10.4 (SCL), U11.4 (SCL), U12.4 (SCL), U13.4 (SCL)
- net I2C1_SDA_TDM: now also U10.3 (SDA), U11.3 (SDA), U12.3 (SDA), U13.3 (SDA)
- net IOR5A_RGBLED: now also J2.1 (Pin_1), J9.1 (Pin_1)
- net VDD_TDM: now also R19.2, U10.7 (IN-), U11.7 (IN-), U12.7 (IN-), U13.7 (IN-)
- net IOT8A: now reaches J2.2 (Pin_2), J9.2 (Pin_2)
- net IOT8B: now reaches J2.3 (Pin_3), J9.3 (Pin_3)
- net IOT10A: now reaches J2.4 (Pin_4), J9.4 (Pin_4)
- net IOT10B: now reaches J2.5 (Pin_5), J9.5 (Pin_5)
- net IOT11A: now reaches J2.6 (Pin_6), J9.6 (Pin_6)
- net IOT11B: now reaches J2.7 (Pin_7), J9.7 (Pin_7)
- net IOT12A: now reaches J2.8 (Pin_8), J9.8 (Pin_8)
- net IOT12B: now reaches J2.9 (Pin_9), J9.9 (Pin_9)
- net at U7.1 (A1): now also U7.2 (A0), J5.1 (Pin_1), J5.2 (Pin_2), R13.2, R14.2
- net at U9.CN10_19 (PC7): now also R19.1, TH1.2
- net TDM_DBG_TX: now reaches U9.CN10_35 (PA2)
- net TDM_DBG_TX: now also J4.1 (Pin_1)
- net TDM_DBG_RX: now reaches U9.CN10_37 (PA3)
- net TDM_DBG_RX: now also J4.2 (Pin_2)
- new net: J6.1 (Pin_1), J6.2 (Pin_2), R20.2, R21.2, U10.1 (A1), U10.2 (A0)
- new net: J10.1 (Pin_1), J10.2 (Pin_2), R23.2, R25.2, U12.1 (A1), U12.2 (A0)
- new net: J11.1 (Pin_1), J11.2 (Pin_2), R26.2, R28.2, U13.1 (A1), U13.2 (A0)
- new net: J7.1 (Pin_1), J7.2 (Pin_2), R22.2, R24.2, U11.1 (A1), U11.2 (A0)
- new net AAM_DBG_RX: J12.2 (Pin_2)
- new net AAM_DBG_TX: J12.1 (Pin_1)
- new net DSM_DBG_RX: J13.2 (Pin_2)
- new net DSM_DBG_TX: J13.1 (Pin_1)
Other:
- note added: "INA219 AAM"
- note added: "INA219 ACM"
- note added: "INA219 DSM"
- note added: "INA219 TDM"
- note added: "INA219 UUM"
- note added: "Telemetry Debug Module"
- moved on the sheet: D1, D2, D3, D4, R11, R12, R15, R16, R17, R18, U3B, U5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

Commit message: more schematic updates. semiworking PCB
Parts:
- added C6: 10uf, Capacitor_SMD:C_0201_0603Metric, symbol Device:C_Small
- added D10, D11, D5, D6, D7, D8, D9: LED_PWR, LED_SMD:LED_Kingbright_KPBD-3224, symbol Device:LED
- added D12: LED_OK, LED_SMD:LED_Kingbright_KPBD-3224, symbol Device:LED
- added D13: LED_FAIL, LED_SMD:LED_Kingbright_KPBD-3224, symbol Device:LED
- added D14: LED_WARN, LED_SMD:LED_Kingbright_KPBD-3224, symbol Device:LED
- added J14: ACM_DBG, Connector_PinHeader_1.00mm:PinHeader_1x03_P1.00mm_Horizontal, symbol Connector_Generic:Conn_01x03
- added R27, R29, R30, R31, R32, R33, R34, R35, R36, R37: 300, Resistor_SMD:R_0805_2012Metric_Pad1.20x1.40mm_HandSolder, symbol Device:R
- added U14: W25Q128JVS, Package_SO:SOIC-8_5.3x5.3mm_P1.27mm, symbol Memory_Flash:W25Q128JVS
- added U15: AP2112K-3.3, Package_TO_SOT_SMD:SOT-23-5, symbol Regulator_Linear:AP2112K-3.3
- added U16: 74HC4050D, 74HC4050D:SO16, symbol 74HC4050D:74HC4050D
Connections:
- net 3V3_ACM: now also U14.3 (~{WP}/IO_{2}), U14.7 (~{HOLD}/~{RESET}/IO_{3}), U16.1 (VCC)
- net 5V_ACM: now also U10.8 (IN+)
- net 5V_TDM: no longer U10.8 (IN+), U11.8 (IN+), U12.8 (IN+), U13.8 (IN+)
- net GND: now also U3.CN10_20 (GND_S2), U3.CN10_9 (GND_S2), C6.2, D10.1 (K), D11.1 (K), D12.1 (K), D13.1 (K), D14.1 (K), D5.1 (K), D6.1 (K), D7.1 (K), D8.1 (K), D9.1 (K), J14.3 (Pin_3), U14.4 (GND), U15.2 (GND), U16.11 (5A), U16.14 (6A), U16.8 (GND)
- net 5V_UUM: now reaches U3.CN10_8 (U5V)
- net 5V_UUM: now also U12.8 (IN+)
- net I2C1_SCL_TDM renamed TDM_I2C1_SCL
- net I2C1_SDA_TDM renamed TDM_I2C1_SDA
- net IOB11A_PMOD2.2 renamed ACM_LED_PWR
- net IOB11B_PMOD2.1 renamed ACM_LED_WARN
- net ACM_LED_WARN: now also R36.2
- net IOB13A_PMOD2.8 renamed ACM_LED_FAIL
- net ACM_LED_FAIL: now also R37.2
- net IOB13B_PMOD2.7 renamed ACM_LED_OK
- net ACM_LED_OK: now also R35.2
- net IOB29B_PMOD1.2 renamed ACM_SPI_SCLK
- net ACM_SPI_SCLK: now also U16.5 (2A)
- net IOB31A_PMOD1.3 renamed ACM_SPI_MOSI
- net ACM_SPI_MOSI: now also U16.7 (3A)
- net IOB31B_PMOD1.4 renamed ACM_SPI_CS
- net ACM_SPI_CS: now also U16.3 (1A)
- net IOB33A_PMOD1.1 renamed ACM_SPI_MISO
- net ACM_SPI_MISO: now also U16.9 (4A)
- net IOB8A_PMOD2.4 renamed ACM_DBG_TX
- net ACM_DBG_TX: now also J14.1 (Pin_1)
- net IOB8B_PMOD2.3 renamed ACM_DBG_RX
- net ACM_DBG_RX: now also J14.2 (Pin_2)
- net LEDFAIL_TDM renamed TDM_LED_FAIL
- net LEDOK_TDM renamed TDM_LED_OK
- net LEDWARN_TDM renamed TDM_LED_WARN
- net VDD_TDM renamed TDM_VDD
- net TDM_VDD: now also R27.2; no longer U10.7 (IN-), U11.7 (IN-), U12.7 (IN-), U13.7 (IN-)
- new net: D7.2 (A), R30.1
- new net: D12.2 (A), R35.1
- new net: D10.2 (A), R33.2
- new net: D13.2 (A), R36.1
- new net: U14.1 (~{CS}), U16.2 (1Y)
- new net: U14.2 (DO/IO_{1}), U16.10 (4Y)
- new net: U14.5 (DI/IO_{0}), U16.6 (3Y)
- new net: U14.6 (CLK), U16.4 (2Y)
- new net: C6.1, R33.1, U14.8 (VCC), U15.5 (VOUT)
- new net: D8.2 (A), R31.1
- new net: D6.2 (A), R29.1
- new net: D11.2 (A), R34.1
- new net: D14.2 (A), R37.1
- new net: D9.2 (A), R32.1
- new net: D5.2 (A), R27.1
- new net 5V_AAM: U13.8 (IN+)
- new net 5V_DSM: U11.8 (IN+)
- new net ACM_VDD: R34.2
- new net VDD_AAM: R30.2, U13.7 (IN-)
- new net VDD_ACM: R29.2, U10.7 (IN-), U15.1 (VIN), U15.3 (EN)
- new net VDD_DSM: R32.2, U11.7 (IN-)
- new net VDD_UUM: R31.2, U12.7 (IN-)
Other:
- note added: "Audio Creation Module"
- note added: "Upload & Update Module"
- note added: "W25Q128 ACM"
- moved on the sheet: C1, C2, C3, C4, C5, D1, D2, D3, D4, J1, J10, J11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

Commit message: more schematic updates. semiworking PCB
Parts:
- added D15: LED_PWR, LED_SMD:LED_Kingbright_KPBD-3224, symbol Device:LED
- added D16: LED_OK, LED_SMD:LED_Kingbright_KPBD-3224, symbol Device:LED
- added D17: LED_FAIL, LED_SMD:LED_Kingbright_KPBD-3224, symbol Device:LED
- added D18: LED_WARN, LED_SMD:LED_Kingbright_KPBD-3224, symbol Device:LED
- added R38, R39, R40, R41: 300, Resistor_SMD:R_0805_2012Metric_Pad1.20x1.40mm_HandSolder, symbol Device:R
Connections:
- net ACM_LED_FAIL: now also R41.2
- net ACM_LED_OK: now also R39.2
- net ACM_LED_WARN: now also R40.2
- net ACM_VDD: now also R38.2
- net GND: now also D15.1 (K), D16.1 (K), D17.1 (K), D18.1 (K)
- new net: D17.2 (A), R40.1
- new net: D15.2 (A), R38.1
- new net: D18.2 (A), R41.1
- new net: D16.2 (A), R39.1
Other:
- note added: "Audio Acquisition Module"
- moved on the sheet: U1A, U4
