File: schematic/signalmesh.kicad_sch (KiCad schematic)
At the start: 131 parts, among them J1 FPGA I/O, J10 INA219_CONFIG, J11 INA219_CONFIG, J12 AAM_DBG, J13 DSM_DBG, J14 ACM_DBG, J15 INA219_CONFIG, J16 DSM_DBG, J17 LCD_display, J2 FPGA I/O, J3 LCD_display, J4 TDM_DBG, J5 INA219_CONFIG, J6 INA219_CONFIG, J7 INA219_CONFIG, J8 FPGA I/O, J9 FPGA I/O, U1 NUCLEO-H753ZI, U10 INA219AxD, U11 INA219AxD, U12 INA219AxD, U13 INA219AxD, U14 W25Q128JVS, U15 AP2112K-3.3, U16 74HC4050D, U17 NUCLEO-H753ZI, U18 HDSP-7503, U19 HDSP-7503, U2 HDSP-7503, U20 INA219AxD, U21 74HC4050D, U22 AP2112K-3.3, U23 W25Q128JVS, U24 74HC4050D, U25 AP2112K-3.3, U26 W25Q128JVS, U27 MCP2551-I-P, U28 74LVC1G3157, U29 MCP2551-I-P, U3 NUCLEO-F303RE, U30 MCP2551-I-P, U31 MCP2551-I-P, U4 YAAJ_BluePill_Part_Like, U5 24LC256-I_SN, U6 BME280, U7 INA219AxD, U8 24LC256-I_SN, U9 NUCLEO-F446RE

Commit message: attempting CAN routing. semi routed pcb
Parts:
- added H1, H2, H5, H6: MountingHole, MountingHole:MountingHole_3.2mm_M3, symbol Mechanical:MountingHole
- added J18: LCD_display, Connector_PinHeader_1.00mm:PinHeader_1x04_P1.00mm_Horizontal, symbol Connector_Generic:Conn_01x04
- U27, U29, U30, U31: symbol Interface_CAN_LIN:MCP2551-I-P -> Interface_CAN_LIN_pos_neg:MCP2551-I-P
- U28: footprint (none) -> SN74LVC1G3157:SC70-6
Connections:
- net GND: now also J18.4 (Pin_4)
- net TDM_I2C1_SCL: now also J18.3 (Pin_3)
- net TDM_I2C1_SDA: now also J18.2 (Pin_2)
- net TDM_VDD: now also J18.1 (Pin_1)
- net CAN-: now reaches R44.2, R47.1, U27.6 (CAN-), U29.6 (CAN-), U30.6 (CAN-), U31.6 (CAN-)
- net CAN+: now reaches R44.1, R47.2, U27.7 (CAN+), U29.7 (CAN+), U30.7 (CAN+), U31.7 (CAN+)
- no-connect marks 9 -> 11

Commit message: progress. might have enough of the vital stuff routed to get the autorouter working for the rest. not sure if it will follow rules though
Parts:
- added J19: AudioJack3, Connector_Audio:Jack_3.5mm_CUI_SJ-3523-SMT_Horizontal, symbol Connector_Audio:AudioJack3
Connections:
- net 7SDD_VDD is gone; now on net 5V_7SDD: R1.2
- net AAM_DAC_L: now also J19.T
- net AAM_DAC_R: now also J19.R
- net GND: now also J19.S
Changed lines of the file:
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@@
 	(wire
 		(pts
+			(xy 265.43 184.15) (xy 283.21 184.15)
+		)
+		(stroke
+			(width 0)
+			(type default)
+		)
+	)
+	(wire
+		(pts
 			(xy 618.49 125.73) (xy 622.3 125.73)
 		)
@@
 		)
 	)
-	(global_label "7SDD_VDD"
+	(global_label "5V_7SDD"
 		(shape input)
 		(at 681.99 346.71 180)
@@
 		)
 		(property "Intersheetrefs" "${INTERSHEET_REFS}"
-			(at 669.4496 346.71 0)
+			(at 670.7801 346.71 0)
 			(effects
 				(font
@@
 		)
 	)
+	(global_label "AAM_DAC_R"
+		(shape bidirectional)
+		(at 265.43 186.69 0)
+		(fields_autoplaced yes)
+		(effects
+			(font
+				(size 1.27 1.27)
+			)
+			(justify left)
+		)
+		(property "Intersheetrefs" "${INTERSHEET_REFS}"
+			(at 279.9889 186.69 0)
+			(effects
+				(font
+					(size 1.27 1.27)
+				)
+				(justify left)
+				(hide yes)
+			)
+		)
+	)
 	(global_label "AAM_FMC_D6"
 		(shape bidirectional)
@@
 		)
 	)
+	(global_label "AAM_DAC_L"
+		(shape bidirectional)
+		(at 265.43 189.23 0)
+		(fields_autoplaced yes)
+		(effects
+			(font
+				(size 1.27 1.27)
+			)
+			(justify left)
+		)
+		(property "Intersheetrefs" "${INTERSHEET_REFS}"
+			(at 279.747 189.23 0)
+			(effects
+				(font
+					(size 1.27 1.27)
+				)
+				(justify left)
+				(hide yes)
+			)
+		)
+	)
 	(global_label "AAM_FMC_D10"
 		(shape bidirectional)
@@
 	)
 	(symbol
+		(lib_id "Connector_Audio:AudioJack3")
+		(at 260.35 186.69 0)
+		(unit 1)
+		(exclude_from_sim no)
+		(in_bom yes)
+		(on_board yes)
+		(dnp no)
+		(fields_autoplaced yes)
+		(property "Reference" "J19"
+			(at 258.445 177.8 0)
+			(effects
+				(font
+					(size 1.27 1.27)
+				)
+			)
+		)
+		(property "Value" "AudioJack3"
+			(at 258.445 180.34 0)
+			(effects
+				(font
+					(size 1.27 1.27)
+				)
+			)
+		)
+		(property "Footprint" "Connector_Audio:Jack_3.5mm_CUI_SJ-3523-SMT_Horizontal"
+			(at 260.35 186.69 0)
+			(effects
+				(font
+					(size 1.27 1.27)
+				)
+				(hide yes)
+			)
+		)
+		(property "Datasheet" "~"
+			(at 260.35 186.69 0)
+			(effects
+				(font
+					(size 1.27 1.27)
+				)
+				(hide yes)
+			)
+		)
+		(property "Description" "Audio Jack, 3 Poles (Stereo / TRS)"
+			(at 260.35 186.69 0)
+			(effects
+				(font
+					(size 1.27 1.27)
+				)
+				(hide yes)
+			)
+		)
+		(pin "T"
+		)
+		(pin "S"
+		)
+		(pin "R"
+		)
+		(instances
+			(project ""
+				(path "/fe7b15e9-f0ed-4338-9f03-dd7651dace13"
+					(reference "J19")
+					(unit 1)
+				)
+			)
+		)
+	)
+	(symbol
 		(lib_id "power:GND")
 		(at 532.13 128.27 0)
@@
 					(unit 1)
 				)
+			)
+		)
+	)
+	(symbol
+		(lib_id "power:GND")
+		(at 283.21 184.15 0)
+		(unit 1)
+		(exclude_from_sim no)
+		(in_bom yes)
+		(on_board yes)
+		(dnp no)
+		(fields_autoplaced yes)
+		(property "Reference" "#PWR0128"
+			(at 283.21 190.5 0)
+			(effects
+				(font
+					(size 1.27 1.27)
+				)
+				(hide yes)
+			)
+		)
+		(property "Value" "GND"
+			(at 283.21 189.23 0)
+			(effects
+				(font
+					(size 1.27 1.27)
+				)
+			)
+		)
+		(property "Footprint" ""
+			(at 283.21 184.15 0)
+			(effects
+				(font
+					(size 1.27 1.27)
+				)
+				(hide yes)
+			)
+		)
+		(property "Datasheet" ""
+			(at 283.21 184.15 0)
+			(effects
+				(font
+					(size 1.27 1.27)
+				)
+				(hide yes)
+			)
+		)
+		(property "Description" "Power symbol creates a global label with name \"GND\" , ground"
+			(at 283.21 184.15 0)
+			(effects
+				(font
+					(size 1.27 1.27)
+				)
+				(hide yes)
+			)
+		)
+		(pin "1"
+		)
+		(instances
+			(project "signalmesh"
+				(path "/fe7b15e9-f0ed-4338-9f03-dd7651dace13"
+					(reference "#PWR0128")
+					(unit 1)
+				)
