File: schematic/signalmesh.kicad_sch (KiCad schematic)
At the start: 137 parts, among them J1 FPGA I/O, J10 INA219_CONFIG, J11 INA219_CONFIG, J12 AAM_DBG, J13 DSM_DBG, J14 ACM_DBG, J15 INA219_CONFIG, J16 DSM_DBG, J17 LCD_display, J18 LCD_display, J19 AudioJack3, J2 FPGA I/O, J3 LCD_display, J4 TDM_DBG, J5 INA219_CONFIG, J6 INA219_CONFIG, J7 INA219_CONFIG, J8 FPGA I/O, J9 FPGA I/O, U1 NUCLEO-H753ZI, U10 INA219AxD, U11 INA219AxD, U12 INA219AxD, U13 INA219AxD, U14 W25Q128JVS, U15 AP2112K-3.3, U16 74HC4050D, U17 NUCLEO-H753ZI, U18 HDSP-7503, U19 HDSP-7503, U2 HDSP-7503, U20 INA219AxD, U21 74HC4050D, U22 AP2112K-3.3, U23 W25Q128JVS, U24 74HC4050D, U25 AP2112K-3.3, U26 W25Q128JVS, U27 MCP2551-I-P, U28 74LVC1G3157, U29 MCP2551-I-P, U3 NUCLEO-F303RE, U30 MCP2551-I-P, U31 MCP2551-I-P, U4 YAAJ_BluePill_Part_Like, U5 24LC256-I_SN, U6 BME280, U7 INA219AxD, U8 24LC256-I_SN, U9 NUCLEO-F446RE

Commit message: ugh routing is a bit messy right now. need to go back to schematic and finish up wiring i forgot about primarily the UARTs for debugging on all boards and the cmd UART from AAM<->ACM
Parts:
- C1, C10, C2, C3, C4, C5, C6, C7, C8, C9: footprint Capacitor_SMD:C_0201_0603Metric -> Capacitor_SMD:C_0805_2012Metric
- D1, D10, D11, D12, D13, D14, D15, D16, D17, D18, D19, D2, D20, D21, D22, D23, D24, D25, D26, D27, D3, D4, D5, D6, D7, D8, D9: footprint LED_SMD:LED_Kingbright_KPBD-3224 -> LED_SMD:LED_0603_1608Metric
Connections:
- net ACM_CMD_RX is gone; now on net AAM_CMD_RX: J1.8 (Pin_8), J8.8 (Pin_8)
- net ACM_CMD_TX is gone; now on net AAM_CMD_RX: J1.7 (Pin_7), J8.7 (Pin_7)
- net AAM_CAN_RD: now also U1.CN12_3 (PB8), U29.1 (TXD); no longer U29.4 (RXD)
- net AAM_CAN_TD: now also U1.CN12_5 (PB9), U29.4 (RXD); no longer U29.1 (TXD)
- net DSM_CAN_RD: now also U17.CN12_3 (PB8), U30.1 (TXD); no longer U30.4 (RXD)
- net DSM_CAN_TD: now also U17.CN12_5 (PB9), U30.4 (RXD); no longer U30.1 (TXD)
- net TDM_CAN_RD: now also U31.1 (TXD), U9.CN10_14 (PA11); no longer U31.4 (RXD)
- net TDM_CAN_TD: now also U31.4 (RXD), U9.CN10_12 (PA12); no longer U31.1 (TXD)
- net UUM_CAN_RD: now also U27.1 (TXD), U3.CN10_14 (PA11); no longer U27.4 (RXD)
- net UUM_CAN_TD: now also U27.4 (RXD), U3.CN10_12 (PA12); no longer U27.1 (TXD)
- net AAM_CMD_RX: now reaches U1.CN11_1 (PC10)
- net AAM_CMD_RX: now also U1.CN11_2 (PC11)
Other:
- note added: "AAM <-> ACM command ctrl"
- moved on the sheet: U17F, U1A, U1C, U1D, U1E, U1F

Commit message: good progress. build from here. bit of autorouter. not too shitty
Parts:
- J13: value DSM_DBG -> UUM_DBG
- J17, J18, J3: footprint Connector_PinHeader_1.00mm:PinHeader_1x04_P1.00mm_Horizontal -> Connector_PinHeader_1.00mm:PinHeader_1x04_P1.00mm_Vertical_SMD_Pin1Left
Connections:
- net AAM_CMD_RX: no longer J1.8 (Pin_8), J8.8 (Pin_8), U1.CN11_1 (PC10)
- net DSM_DBG_RX: no longer J13.2 (Pin_2)
- net DSM_DBG_TX: no longer J13.1 (Pin_1)
- net UUM_DBG_RX: now also J13.2 (Pin_2)
- net UUM_DBG_TX: now also J13.1 (Pin_1)
- net UUM_SPI1_CS: no longer U24.3 (1A)
- net UUM_SPI2_CS: now reaches U3.CN10_21 (PA9)
- net UUM_SPI2_CS: now also U24.3 (1A)
- new net AAM_CMD_TX: J1.8 (Pin_8), J8.8 (Pin_8), U1.CN11_1 (PC10)
Other:
- note added: "AAM <-> ACM cmd ctrl"
- note removed: "AAM <-> ACM command ctrl"
- moved on the sheet: C10, C8, C9, D25, D26, R10, R42, R9, U21, U22, U23, U24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

Commit message: adding JLCPCB files
Parts:
- added D28: LED_PWR, LED_SMD:LED_0603_1608Metric, symbol Device:LED
- added D29: LED_OK, LED_SMD:LED_0603_1608Metric, symbol Device:LED
- added D30: LED_FAIL, LED_SMD:LED_0603_1608Metric, symbol Device:LED
- added D31: LED_WARN, LED_SMD:LED_0603_1608Metric, symbol Device:LED
- added R45, R46, R48, R49: 300, Resistor_SMD:R_0805_2012Metric_Pad1.20x1.40mm_HandSolder, symbol Device:R
Connections:
- net AAM_LED_FAIL: now also U1.CN12_34 (PC4)
- net AAM_LED_OK: now also U1.CN12_4 (PC6)
- net AAM_LED_WARN: now also U1.CN12_6 (PC5)
- net DSM_LED_FAIL: now also U17.CN12_34 (PC4)
- net DSM_LED_OK: now also U17.CN12_4 (PC6)
- net DSM_LED_WARN: now also U17.CN12_6 (PC5)
- net GND: now also D28.1 (K), D29.1 (K), D30.1 (K), D31.1 (K)
- net UUM_LED_OK: now reaches U3.CN7_35 (PC2)
- net UUM_LED_OK: now also R46.2
- net UUM_LED_WARN: now reaches U3.CN7_36 (PC1)
- net UUM_LED_WARN: now also R48.2
- net UUM_LED_FAIL: now reaches U3.CN7_38 (PC0)
- net UUM_LED_FAIL: now also R49.2
- new net: D29.2 (A), R46.1
- new net: D28.2 (A), R45.1
- new net: D31.2 (A), R49.1
- new net: D30.2 (A), R48.1
- new net UUM_VDD: R45.2
Other:
- moved on the sheet: U1E
