File: schematic/_autosave-signalmesh.kicad_sch (KiCad schematic)
At the start: 85 parts, among them J1 FPGA I/O, J10 INA219_CONFIG, J11 INA219_CONFIG, J12 AAM_DBG, J13 DSM_DBG, J14 ACM_DBG, J2 FPGA I/O, J4 TDM_DBG, J5 INA219_CONFIG, J6 INA219_CONFIG, J7 INA219_CONFIG, J8 FPGA I/O, J9 FPGA I/O, U1 NUCLEO-H753ZI, U10 INA219AxD, U11 INA219AxD, U12 INA219AxD, U13 INA219AxD, U14 W25Q128JVS, U15 AP2112K-3.3, U16 74HC4050D, U2 NUCLEO-H753ZI, U3 NUCLEO-F303RE, U4 YAAJ_BluePill_Part_Like, U5 24LC256-I_SN, U6 BME280, U7 INA219AxD, U8 24LC256-I_SN, U9 NUCLEO-F446RE

Commit message: attempt at FMC interface
Connections:
- net ACM_FMC_D10 renamed AAM_FMC_D10
- net ACM_FMC_D11 renamed AAM_FMC_D11
- net ACM_FMC_D12 renamed AAM_FMC_D12
- net ACM_FMC_D13 renamed AAM_FMC_D13
- net ACM_FMC_D8 renamed AAM_FMC_D8
- net ACM_FMC_D9 renamed AAM_FMC_D9
Other:
- moved on the sheet: D15, D16, D17, D18, R38, R39, R40, R41, U1A, U1B, U1C, U1D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
