File: schematic/signalmesh.kicad_pcb (KiCad board)
At the start: 2 copper layers, 536 x 151 mm, 24 parts, among them J1 FPGA I/O, J2 FPGA I/O, J8 FPGA I/O, J9 FPGA I/O, U1 NUCLEO-H753ZI, U2 NUCLEO-H753ZI, U3 NUCLEO-F303RE, U4 YAAJ_BluePill_Part_Like, U5 24LC256-I_SN, U6 BME280, U7 INA219AxD, U8 24LC256-I_SN, U9 NUCLEO-F446RE

Commit message: update schematic and pcb. errors
Parts:
- removed R10: 300, Resistor_SMD:R_0805_2012Metric_Pad1.20x1.40mm_HandSolder
- added C1: 0.1uf, Capacitor_SMD:C_0201_0603Metric, F.Cu at (548.2, 169.0)
- added C2: 0.1uf, Capacitor_SMD:C_0201_0603Metric, F.Cu at (547.9, 175.5)
- added C3: 0.1uf, Capacitor_SMD:C_0201_0603Metric, F.Cu at (548.0, 182.0)
- added C4: 0.1uf, Capacitor_SMD:C_0201_0603Metric, F.Cu at (548.0, 188.8)
- added C5: 0.1uf, Capacitor_SMD:C_0201_0603Metric, F.Cu at (548.0, 195.5)
- added J10: INA219_CONFIG, Connector_PinHeader_1.00mm:PinHeader_1x02_P1.00mm_Horizontal, F.Cu at (556.4, 186.5)
- added J11: INA219_CONFIG, Connector_PinHeader_1.00mm:PinHeader_1x02_P1.00mm_Horizontal, F.Cu at (556.4, 192.5)
- added J4: TDM_DBG, Connector_PinHeader_1.00mm:PinHeader_1x03_P1.00mm_Horizontal, F.Cu at (343.0, 53.9)
- added J5: INA219_CONFIG, Connector_PinHeader_1.00mm:PinHeader_1x02_P1.00mm_Horizontal, F.Cu at (556.4, 167.0)
- added J6: INA219_CONFIG, Connector_PinHeader_1.00mm:PinHeader_1x02_P1.00mm_Horizontal, F.Cu at (556.4, 173.5)
- added J7: INA219_CONFIG, Connector_PinHeader_1.00mm:PinHeader_1x02_P1.00mm_Horizontal, F.Cu at (556.4, 180.3)
- added R13: 10k, Resistor_SMD:R_0805_2012Metric_Pad1.20x1.40mm_HandSolder, F.Cu at (551.2, 165.5)
- added R14: 10k, Resistor_SMD:R_0805_2012Metric_Pad1.20x1.40mm_HandSolder, F.Cu at (551.2, 168.4)
- added R19: 10k, Resistor_SMD:R_0805_2012Metric_Pad1.20x1.40mm_HandSolder, F.Cu at (558.5, 143.5)
- added R20: 10k, Resistor_SMD:R_0805_2012Metric_Pad1.20x1.40mm_HandSolder, F.Cu at (551.2, 172.1)
- added R21: 10k, Resistor_SMD:R_0805_2012Metric_Pad1.20x1.40mm_HandSolder, F.Cu at (551.2, 175.0)
- added R22: 10k, Resistor_SMD:R_0805_2012Metric_Pad1.20x1.40mm_HandSolder, F.Cu at (551.2, 178.6)
- added R23: 10k, Resistor_SMD:R_0805_2012Metric_Pad1.20x1.40mm_HandSolder, F.Cu at (551.2, 185.5)
- added R24: 10k, Resistor_SMD:R_0805_2012Metric_Pad1.20x1.40mm_HandSolder, F.Cu at (551.2, 181.7)
- added R25: 10k, Resistor_SMD:R_0805_2012Metric_Pad1.20x1.40mm_HandSolder, F.Cu at (551.2, 188.2)
- added R26: 10k, Resistor_SMD:R_0805_2012Metric_Pad1.20x1.40mm_HandSolder, F.Cu at (551.2, 192.0)
- added R28: 10k, Resistor_SMD:R_0805_2012Metric_Pad1.20x1.40mm_HandSolder, F.Cu at (551.2, 194.9)
- added TH1: 10k, OptoDevice:R_LDR_4.9x4.2mm_P2.54mm_Vertical, F.Cu at (551.5, 143.5)
- added U10: INA219AxD, Package_SO:SOIC-8_3.9x4.9mm_P1.27mm, F.Cu at (543.2, 173.6)
- added U11: INA219AxD, Package_SO:SOIC-8_3.9x4.9mm_P1.27mm, F.Cu at (543.2, 180.2)
- added U12: INA219AxD, Package_SO:SOIC-8_3.9x4.9mm_P1.27mm, F.Cu at (543.2, 186.7)
- added U13: INA219AxD, Package_SO:SOIC-8_3.9x4.9mm_P1.27mm, F.Cu at (543.2, 193.3)
- moved U4 413.4 mm to (449.2, 143.1), turned to 0 degrees
- moved U6 228.3 mm to (300.0, 185.0)
- moved U5 35.0 mm to (526.0, 155.4)
- moved U7 21.4 mm to (543.3, 167.0)
- moved R11 19.0 mm to (550.0, 153.0), turned to 90 degrees
- moved R12 17.5 mm to (555.5, 153.0), turned to 90 degrees
- moved R15 16.6 mm to (499.8, 157.7), turned to 180 degrees
- moved R18 15.6 mm to (499.8, 153.7), turned to 180 degrees
- moved D1 15.4 mm to (507.8, 145.1), turned to -90 degrees
- moved U8 14.8 mm to (526.0, 147.5)
- moved D4 13.0 mm to (507.7, 157.8), turned to -90 degrees
- moved D2 11.9 mm to (507.7, 149.3), turned to -90 degrees
- moved D3 10.9 mm to (507.7, 153.5), turned to -90 degrees
- moved R16 10.1 mm to (499.8, 145.1), turned to 180 degrees
- moved R17 4.49 mm to (499.8, 149.6), turned to 180 degrees
Connections:
- net Net-(J2-Pin_1) renamed IOR5A_RGBLED
- net Net-(J2-Pin_2) renamed IOT8A
- net Net-(J2-Pin_3) renamed IOT8B
- net Net-(J2-Pin_4) renamed IOT10A
- net Net-(J2-Pin_5) renamed IOT10B
- net Net-(J2-Pin_6) renamed IOT11A
- net Net-(J2-Pin_7) renamed IOT11B
- net Net-(J2-Pin_8) renamed IOT12A
- net Net-(J2-Pin_9) renamed IOT12B
- U7 pad 1: unconnected-(U7-A1-Pad1) -> Net-(J5-Pin_1)
- U7 pad 2: unconnected-(U7-A0-Pad2) -> Net-(J5-Pin_1)
- U8 pad 2: GND -> unconnected-(U8-A1-Pad2)
- U9 pad CN10_19: unconnected-(U9B-PC7-PadCN10_19) -> Net-(U9B-PC7)
- U9 pad CN10_35: unconnected-(U9B-PA2-PadCN10_35) -> TDM_DBG_TX
- U9 pad CN10_37: unconnected-(U9B-PA3-PadCN10_37) -> TDM_DBG_RX
Routing:
- net I2C1_SCL_TDM: track 0.00 -> 418.0 mm, vias 0 -> 6
- net I2C1_SDA_TDM: track 0.00 -> 408.3 mm, vias 0 -> 7
- net VDD_TDM: track 0.00 -> 390.7 mm, vias 0 -> 5
- net TDM_DBG_RX: track 0.00 -> 281.1 mm, vias 0 -> 1
- net TDM_DBG_TX: track 0.00 -> 281.0 mm, vias 0 -> 1
- net 5V_TDM: track 0.00 -> 154.8 mm, vias 0 -> 6
- net LEDFAIL_TDM: track 0.00 -> 112.5 mm, vias 0 -> 2
- net LEDOK_TDM: track 0.00 -> 94.5 mm, vias 0 -> 2
- net Net-(U1A-GND_CN11-PadCN11_19): track 0.00 -> 91.7 mm
- net Net-(U2A-GND_CN11-PadCN11_19): track 0.00 -> 90.4 mm
- net LEDWARN_TDM: track 0.00 -> 74.4 mm, vias 0 -> 1
- net GND: track 0.00 -> 63.2 mm, vias 0 -> 26
- net Net-(U9B-PC7): track 0.00 -> 48.6 mm
- net Net-(J7-Pin_1): track 0.00 -> 24.1 mm
- net Net-(J10-Pin_1): track 0.00 -> 23.7 mm
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- added copper zone on B.Cu, net GND
Other:
- outline, holes or cut-outs redrawn
- board text added: "Crash Table"
- board text added: "FAIL"
- board text added: "I2C"
- board text added: "OK"
- board text added: "PWR"
- board text added: "Power Monitor"
- board text added: "TDM_DBG"
- board text added: "WARN"

Commit message: more schematic updates. semiworking PCB
Parts:
- added D5: LED_PWR, LED_SMD:LED_Kingbright_KPBD-3224, F.Cu at (531.0, 166.8)
- added D6: LED_PWR, LED_SMD:LED_Kingbright_KPBD-3224, F.Cu at (531.0, 173.2)
- added D7: LED_PWR, LED_SMD:LED_Kingbright_KPBD-3224, F.Cu at (531.0, 192.7)
- added D8: LED_PWR, LED_SMD:LED_Kingbright_KPBD-3224, F.Cu at (531.0, 186.2)
- added D9: LED_PWR, LED_SMD:LED_Kingbright_KPBD-3224, F.Cu at (531.0, 179.7)
- added J12: AAM_DBG, Connector_PinHeader_1.00mm:PinHeader_1x03_P1.00mm_Horizontal, F.Cu at (365.0, 53.9)
- added J13: DSM_DBG, Connector_PinHeader_1.00mm:PinHeader_1x03_P1.00mm_Horizontal, F.Cu at (377.5, 53.9)
- added R27: 300, Resistor_SMD:R_0805_2012Metric_Pad1.20x1.40mm_HandSolder, F.Cu at (536.5, 166.8)
- added R29: 300, Resistor_SMD:R_0805_2012Metric_Pad1.20x1.40mm_HandSolder, F.Cu at (536.5, 173.2)
- added R30: 300, Resistor_SMD:R_0805_2012Metric_Pad1.20x1.40mm_HandSolder, F.Cu at (536.5, 192.5)
- added R31: 300, Resistor_SMD:R_0805_2012Metric_Pad1.20x1.40mm_HandSolder, F.Cu at (536.5, 186.1)
- added R32: 300, Resistor_SMD:R_0805_2012Metric_Pad1.20x1.40mm_HandSolder, F.Cu at (536.5, 179.6)
- moved U4 247.1 mm to (207.7, 90.7), turned to 90 degrees
- moved U3 157.1 mm to (231.9, 140.5)
- moved U1 113.5 mm to (313.4, 126.5)
- moved J2 80.0 mm to (392.0, 91.5)
- moved J9 80.0 mm to (401.0, 91.5)
- moved J1 79.7 mm to (368.7, 91.5)
- moved J8 79.7 mm to (359.7, 91.5)
- moved U6 79.7 mm to (379.7, 185.0)
- moved U2 47.6 mm to (448.0, 126.8)
- moved J4 47.0 mm to (390.0, 53.9)
- moved R19 9.96 mm to (548.5, 143.5)
- moved TH1 9.96 mm to (541.5, 143.5)
- moved R23 0.90 mm to (552.0, 185.0)
- moved R13 0.75 mm to (552.0, 165.5)
- moved R20 0.75 mm to (552.0, 172.1)
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Connections:
- U10 pad 7: VDD_TDM -> VDD_ACM
- U10 pad 8: 5V_TDM -> 5V_ACM
- U11 pad 7: VDD_TDM -> VDD_DSM
- U11 pad 8: 5V_TDM -> 5V_DSM
- U12 pad 7: VDD_TDM -> VDD_UUM
- U12 pad 8: 5V_TDM -> 5V_UUM
- U13 pad 7: VDD_TDM -> VDD_AAM
- U13 pad 8: 5V_TDM -> 5V_AAM
Routing:
- net VDD_TDM: track 390.7 -> 362.0 mm, vias 5 -> 7
- net GND: track 63.2 -> 76.4 mm, vias 26 -> 31
- net TDM_DBG_TX: track 281.0 -> 278.0 mm
- net Net-(J10-Pin_1): track 23.7 -> 26.6 mm
- net IOB13B_PMOD2.7: track 9.00 -> 11.5 mm
- net TDM_DBG_RX: track 281.1 -> 278.7 mm
- net I2C1_SCL_TDM: track 418.0 -> 420.4 mm
- net Net-(U9B-PC7): track 48.6 -> 50.8 mm
- net I2C1_SDA_TDM: track 408.3 -> 410.4 mm, vias 7 -> 1
- net Net-(U2A-GND_CN11-PadCN11_19): track 90.4 -> 88.9 mm
- net LEDOK_TDM: track 94.5 -> 95.8 mm, vias 2 -> 1
Other:
- board text added: "AAM_DBG"
- board text added: "ACM_DBG"
- board text added: "GND"
- board text added: "RX"
- board text added: "TX"

Commit message: attempt at FMC interface
Parts:
- added C6: 10uf, Capacitor_SMD:C_0201_0603Metric, F.Cu at (410.1, 168.5)
- added D10: LED_PWR, LED_SMD:LED_Kingbright_KPBD-3224, F.Cu at (404.0, 171.5)
- added D11: LED_PWR, LED_SMD:LED_Kingbright_KPBD-3224, F.Cu at (366.3, 175.0)
- added D12: LED_OK, LED_SMD:LED_Kingbright_KPBD-3224, F.Cu at (366.3, 179.3)
- added D13: LED_FAIL, LED_SMD:LED_Kingbright_KPBD-3224, F.Cu at (366.2, 183.7)
- added D14: LED_WARN, LED_SMD:LED_Kingbright_KPBD-3224, F.Cu at (366.2, 188.1)
- added D15: LED_PWR, LED_SMD:LED_Kingbright_KPBD-3224, F.Cu at (363.0, 66.5)
- added D16: LED_OK, LED_SMD:LED_Kingbright_KPBD-3224, F.Cu at (362.8, 81.0)
- added D17: LED_FAIL, LED_SMD:LED_Kingbright_KPBD-3224, F.Cu at (362.8, 75.7)
- added D18: LED_WARN, LED_SMD:LED_Kingbright_KPBD-3224, F.Cu at (363.0, 71.0)
- added J14: ACM_DBG, Connector_PinHeader_1.00mm:PinHeader_1x03_P1.00mm_Horizontal, F.Cu at (362.4, 53.8)
- added R33: 300, Resistor_SMD:R_0805_2012Metric_Pad1.20x1.40mm_HandSolder, F.Cu at (404.0, 167.5)
- added R34: 300, Resistor_SMD:R_0805_2012Metric_Pad1.20x1.40mm_HandSolder, F.Cu at (358.0, 175.3)
- added R35: 300, Resistor_SMD:R_0805_2012Metric_Pad1.20x1.40mm_HandSolder, F.Cu at (358.1, 179.5)
- added R36: 300, Resistor_SMD:R_0805_2012Metric_Pad1.20x1.40mm_HandSolder, F.Cu at (358.0, 183.7)
- added R37: 300, Resistor_SMD:R_0805_2012Metric_Pad1.20x1.40mm_HandSolder, F.Cu at (358.0, 187.9)
- added R38: 300, Resistor_SMD:R_0805_2012Metric_Pad1.20x1.40mm_HandSolder, F.Cu at (356.0, 67.0)
- added R39: 300, Resistor_SMD:R_0805_2012Metric_Pad1.20x1.40mm_HandSolder, F.Cu at (356.2, 81.2)
- added R40: 300, Resistor_SMD:R_0805_2012Metric_Pad1.20x1.40mm_HandSolder, F.Cu at (356.2, 76.0)
- added R41: 300, Resistor_SMD:R_0805_2012Metric_Pad1.20x1.40mm_HandSolder, F.Cu at (356.2, 71.2)
- added U14: W25Q128JVS, Package_SO:SOIC-8_5.3x5.3mm_P1.27mm, F.Cu at (388.5, 178.6)
- added U15: AP2112K-3.3, Package_TO_SOT_SMD:SOT-23-5, F.Cu at (398.3, 168.4)
- added U16: 74HC4050D, 74HC4050D:SO16, F.Cu at (400.9, 178.5)
- moved U4 17.9 mm to (207.1, 72.8)
- moved U3 14.1 mm to (230.3, 154.5)
- moved TH1 12.7 mm to (553.7, 139.6), turned to 0 degrees
- moved U5 12.6 mm to (538.6, 155.5)
- moved U8 12.6 mm to (538.6, 147.6)
- moved D1 12.6 mm to (520.4, 145.2)
- moved D2 12.6 mm to (520.3, 149.4)
- moved D3 12.6 mm to (520.3, 153.6)
- moved D4 12.6 mm to (520.3, 157.9)
- moved R15 12.6 mm to (512.4, 157.8)
- moved R16 12.6 mm to (512.4, 145.2)
- moved R17 12.6 mm to (512.4, 149.7)
- moved R18 12.6 mm to (512.4, 153.8)
- moved U6 11.5 mm to (379.7, 196.5)
- moved J1 11.5 mm to (368.7, 103.0)
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Connections:
- net I2C1_SCL_TDM renamed TDM_I2C1_SCL
- net I2C1_SDA_TDM renamed TDM_I2C1_SDA
- net IOB11A_PMOD2.2 renamed ACM_CMD_TX
- net IOB11B_PMOD2.1 renamed ACM_CMD_RX
- net IOB13A_PMOD2.8 renamed ACM_LED_PWR
- net IOB13B_PMOD2.7 renamed ACM_LED_WARN
- net IOB15A_PMOD4.2 renamed AAM_FMC_A8
- net IOB15B_PMOD4.1 renamed AAM_FMC_A9
- net IOB23A_PMOD2.6 renamed ACM_LED_FAIL
- net IOB23B_PMOD2.5 renamed ACM_LED_OK
- net IOB29A_PMOD3.3 renamed AAM_FMC_A11
- net IOB29B_PMOD1.2 renamed ACM_SPI_SCLK
- net IOB31A_PMOD1.3 renamed ACM_SPI_MOSI
- net IOB31B_PMOD1.4 renamed ACM_SPI_CS
- net IOB33A_PMOD1.1 renamed ACM_SPI_MISO
- net IOB33B_PMOD3.4 renamed AAM_FMC_A10
- net IOB41A_PMOD3.2 renamed AAM_FMC_A12
- net IOB41B_PMOD3.1 renamed AAM_FMC_A13
- net IOB8A_PMOD2.4 renamed ACM_DBG_TX
- net IOB8B_PMOD2.3 renamed ACM_DBG_RX
- net IOR15B_PMOD3.7 renamed AAM_FMC_A15
- net IOR17B_PMOD3.8 renamed AAM_FMC_A14
- net IOR24A_PMOD1.5 renamed AAM_FMC_A7
- net IOR24B_PMOD1.6 renamed AAM_FMC_A6
- net LEDFAIL_TDM renamed TDM_LED_FAIL
- net LEDOK_TDM renamed TDM_LED_OK
- net LEDWARN_TDM renamed TDM_LED_WARN
- net VDD_TDM renamed TDM_VDD
- J1 pad 19: IOR15A_PMOD3.6 -> unconnected-(J1-Pin_19-Pad19)
- J1 pad 20: IOR14B_PMOD3.5 -> unconnected-(J1-Pin_20-Pad20)
- J1 pad 21: IOR14A_PMOD4.4 -> unconnected-(J1-Pin_21-Pad21)
- J1 pad 22: IOR13A_PMOD4.3 -> unconnected-(J1-Pin_22-Pad22)
- J2 pad 1: IOR5A_RGBLED -> AAM_FMC_NWE
- J2 pad 10: IOT37A_PMOD1.8 -> AAM_FMC_D6
- J2 pad 11: IOT37B_PMOD1.7 -> AAM_FMC_D7
- J2 pad 12: unconnected-(J2-Pin_12-Pad12) -> AAM_FMC_A0
- J2 pad 13: unconnected-(J2-Pin_13-Pad13) -> AAM_FMC_A1
- J2 pad 14: unconnected-(J2-Pin_14-Pad14) -> AAM_FMC_A2
- J2 pad 15: unconnected-(J2-Pin_15-Pad15) -> AAM_FMC_A3
- J2 pad 16: unconnected-(J2-Pin_16-Pad16) -> AAM_FMC_A4
- J2 pad 2: IOT8A -> AAM_FMC_NOE
- J2 pad 3: IOT8B -> AAM_FMC_NCE
- J2 pad 4: IOT10A -> AAM_FMC_D0
- J2 pad 5: IOT10B -> AAM_FMC_D1
- J2 pad 6: IOT11A -> AAM_FMC_D2
- J2 pad 7: IOT11B -> AAM_FMC_D3
- J2 pad 8: IOT12A -> AAM_FMC_D4
- J2 pad 9: IOT12B -> AAM_FMC_D5
- J8 pad 19: IOR15A_PMOD3.6 -> unconnected-(J8-Pin_19-Pad19)
- J8 pad 20: IOR14B_PMOD3.5 -> unconnected-(J8-Pin_20-Pad20)
- J8 pad 21: IOR14A_PMOD4.4 -> unconnected-(J8-Pin_21-Pad21)
- J8 pad 22: IOR13A_PMOD4.3 -> unconnected-(J8-Pin_22-Pad22)
- J9 pad 1: IOR5A_RGBLED -> AAM_FMC_NWE
- J9 pad 10: IOT37A_PMOD1.8 -> AAM_FMC_D6
- J9 pad 11: IOT37B_PMOD1.7 -> AAM_FMC_D7
- J9 pad 12: unconnected-(J9-Pin_12-Pad12) -> AAM_FMC_A0
- J9 pad 13: unconnected-(J9-Pin_13-Pad13) -> AAM_FMC_A1
- J9 pad 14: unconnected-(J9-Pin_14-Pad14) -> AAM_FMC_A2
- J9 pad 15: unconnected-(J9-Pin_15-Pad15) -> AAM_FMC_A3
- J9 pad 16: unconnected-(J9-Pin_16-Pad16) -> AAM_FMC_A4
- J9 pad 17: unconnected-(J9-Pin_17-Pad17) -> AAM_FMC_A5
- J9 pad 2: IOT8A -> AAM_FMC_NOE
- J9 pad 3: IOT8B -> AAM_FMC_NCE
- J9 pad 4: IOT10A -> AAM_FMC_D0
- J9 pad 5: IOT10B -> AAM_FMC_D1
- J9 pad 6: IOT11A -> AAM_FMC_D2
- J9 pad 7: IOT11B -> AAM_FMC_D3
- J9 pad 8: IOT12A -> AAM_FMC_D4
- J9 pad 9: IOT12B -> AAM_FMC_D5
- U1 pad CN10_1: (no net) -> unconnected-(U1F-AVDD-PadCN10_1)
- U1 pad CN10_10: (no net) -> unconnected-(U1F-D3/TIMER_A_PWM3-PadCN10_10)
- U1 pad CN10_11: (no net) -> unconnected-(U1F-A8/ADC_C_IN-PadCN10_11)
- U1 pad CN10_12: (no net) -> unconnected-(U1F-D2/IO-PadCN10_12)
- U1 pad CN10_13: (no net) -> unconnected-(U1F-D26/QSPI_CS-PadCN10_13)
- U1 pad CN10_14: (no net) -> unconnected-(U1F-D1/USART_A_TX-PadCN10_14)
- U1 pad CN10_15: (no net) -> unconnected-(U1F-D27/QSPI_CLK-PadCN10_15)
- U1 pad CN10_16: (no net) -> AAM_FMC_D4
- U1 pad CN10_17: (no net) -> Net-(U1F-GND_CN10-PadCN10_17)
- U1 pad CN10_18: (no net) -> AAM_FMC_D5
- U1 pad CN10_19: (no net) -> unconnected-(U1F-D28/QSPI_BK1_IO3-PadCN10_19)
- U1 pad CN10_2: (no net) -> unconnected-(U1F-D7/IO-PadCN10_2)
- U1 pad CN10_20: (no net) -> AAM_FMC_D4
- U1 pad CN10_21: (no net) -> unconnected-(U1F-D29/QSPI_BK1_IO1-PadCN10_21)
- U1 pad CN10_22: (no net) -> Net-(U1F-GND_CN10-PadCN10_17)
- U1 pad CN10_23: (no net) -> unconnected-(U1F-D30/QSPI_BK1_IO0-PadCN10_23)
- U1 pad CN10_24: (no net) -> AAM_FMC_D7
- U1 pad CN10_25: (no net) -> unconnected-(U1F-D31/QSPI_BK1_IO2-PadCN10_25)
- U1 pad CN10_26: (no net) -> unconnected-(U1F-D39/TIMER_A_PWM3N-PadCN10_26)
- U1 pad CN10_27: (no net) -> Net-(U1F-GND_CN10-PadCN10_17)
- U1 pad CN10_28: (no net) -> unconnected-(U1F-D38/TIMER_A_BKIN2-PadCN10_28)
- U1 pad CN10_29: (no net) -> unconnected-(U1F-D32/TIMER_C_PWM1-PadCN10_29)
- U1 pad CN10_3: (no net) -> unconnected-(U1F-AGND_CN10-PadCN10_3)
- U1 pad CN10_30: (no net) -> unconnected-(U1F-D37/TIMER_A_BKIN1-PadCN10_30)
- U1 pad CN10_31: (no net) -> unconnected-(U1F-D33/TIMER_D_PWM1-PadCN10_31)
- U1 pad CN10_32: (no net) -> unconnected-(U1F-D36/TIMER_C_PWM2-PadCN10_32)
- U1 pad CN10_33: (no net) -> unconnected-(U1F-D34/TIMER_B_ETR-PadCN10_33)
- U1 pad CN10_34: (no net) -> unconnected-(U1F-D35/TIMER_C_PWM3-PadCN10_34)
- U1 pad CN10_4: (no net) -> AAM_FMC_D6
- U1 pad CN10_5: (no net) -> Net-(U1F-GND_CN10-PadCN10_17)
- U1 pad CN10_6: (no net) -> unconnected-(U1F-D5/TIMER_A_PWM2-PadCN10_6)
- U1 pad CN10_7: (no net) -> unconnected-(U1F-A6/ADC_A_IN-PadCN10_7)
- U1 pad CN10_8: (no net) -> unconnected-(U1F-D4/IO-PadCN10_8)
- U1 pad CN10_9: (no net) -> unconnected-(U1F-A7/ADC_B_IN-PadCN10_9)
- U1 pad CN12_1: (no net) -> unconnected-(U1B-PC9-PadCN12_1)
- U1 pad CN12_10: (no net) -> unconnected-(U1B-PD8-PadCN12_10)
- U1 pad CN12_11: (no net) -> unconnected-(U1B-PA5-PadCN12_11)
- U1 pad CN12_12: (no net) -> unconnected-(U1B-PA12-PadCN12_12)
- U1 pad CN12_13: (no net) -> unconnected-(U1B-PA6-PadCN12_13)
- U1 pad CN12_14: (no net) -> unconnected-(U1B-PA11-PadCN12_14)
- U1 pad CN12_15: (no net) -> unconnected-(U1B-PA7-PadCN12_15)
- U1 pad CN12_16: (no net) -> unconnected-(U1B-PB12-PadCN12_16)
- U1 pad CN12_17: (no net) -> unconnected-(U1B-PB6-PadCN12_17)
- U1 pad CN12_18: (no net) -> unconnected-(U1B-PB11-PadCN12_18)
- U1 pad CN12_19: (no net) -> AAM_FMC_NCE
- U1 pad CN12_2: (no net) -> unconnected-(U1B-PC8-PadCN12_2)
- U1 pad CN12_20: (no net) -> Net-(U1B-GND_CN12-PadCN12_20)
- U1 pad CN12_21: (no net) -> unconnected-(U1B-PA9-PadCN12_21)
- U1 pad CN12_22: (no net) -> unconnected-(U1B-PB2-PadCN12_22)
- U1 pad CN12_23: (no net) -> unconnected-(U1B-PA8-PadCN12_23)
- U1 pad CN12_24: (no net) -> unconnected-(U1B-PB1-PadCN12_24)
- U1 pad CN12_25: (no net) -> unconnected-(U1B-PB10-PadCN12_25)
- U1 pad CN12_26: (no net) -> unconnected-(U1B-PB15-PadCN12_26)
- U1 pad CN12_27: (no net) -> unconnected-(U1B-PB4-PadCN12_27)
- U1 pad CN12_28: (no net) -> unconnected-(U1B-PB14-PadCN12_28)
- U1 pad CN12_29: (no net) -> unconnected-(U1B-PB5-PadCN12_29)
- U1 pad CN12_3: (no net) -> unconnected-(U1B-PB8-PadCN12_3)
- U1 pad CN12_30: (no net) -> unconnected-(U1B-PB13-PadCN12_30)
- U1 pad CN12_31: (no net) -> unconnected-(U1B-PB3-PadCN12_31)
- U1 pad CN12_32: (no net) -> unconnected-(U1B-AGND_CN12-PadCN12_32)
- U1 pad CN12_33: (no net) -> unconnected-(U1B-PA10-PadCN12_33)
- U1 pad CN12_34: (no net) -> unconnected-(U1B-PC4-PadCN12_34)
- U1 pad CN12_35: (no net) -> unconnected-(U1B-PA2-PadCN12_35)
- U1 pad CN12_36: (no net) -> unconnected-(U1B-PF5-PadCN12_36)
- U1 pad CN12_37: (no net) -> unconnected-(U1B-PA3-PadCN12_37)
- U1 pad CN12_38: (no net) -> unconnected-(U1B-PF4-PadCN12_38)
- U1 pad CN12_39: (no net) -> Net-(U1B-GND_CN12-PadCN12_20)
- U1 pad CN12_4: (no net) -> unconnected-(U1B-PC6-PadCN12_4)
- U1 pad CN12_40: (no net) -> unconnected-(U1B-PE8-PadCN12_40)
- U1 pad CN12_41: (no net) -> unconnected-(U1B-PD13-PadCN12_41)
- U1 pad CN12_42: (no net) -> unconnected-(U1B-PF10-PadCN12_42)
- U1 pad CN12_43: (no net) -> unconnected-(U1B-PD12-PadCN12_43)
- U1 pad CN12_44: (no net) -> unconnected-(U1B-PE7-PadCN12_44)
- U1 pad CN12_45: (no net) -> unconnected-(U1B-PD11-PadCN12_45)
- U1 pad CN12_46: (no net) -> unconnected-(U1B-PD14-PadCN12_46)
- U1 pad CN12_47: (no net) -> unconnected-(U1B-PE10-PadCN12_47)
- U1 pad CN12_48: (no net) -> unconnected-(U1B-PD15-PadCN12_48)
- U1 pad CN12_49: (no net) -> unconnected-(U1B-PE12-PadCN12_49)
- U1 pad CN12_5: (no net) -> unconnected-(U1B-PB9-PadCN12_5)
- U1 pad CN12_50: (no net) -> unconnected-(U1B-PF14-PadCN12_50)
- U1 pad CN12_51: (no net) -> unconnected-(U1B-PE14-PadCN12_51)
- U1 pad CN12_52: (no net) -> unconnected-(U1B-PE9-PadCN12_52)
- U1 pad CN12_53: (no net) -> unconnected-(U1B-PE15-PadCN12_53)
- U1 pad CN12_54: (no net) -> Net-(U1B-GND_CN12-PadCN12_20)
- U1 pad CN12_55: (no net) -> unconnected-(U1B-PE13-PadCN12_55)
- U1 pad CN12_56: (no net) -> unconnected-(U1B-PE11-PadCN12_56)
- U1 pad CN12_57: (no net) -> unconnected-(U1B-PF13-PadCN12_57)
- U1 pad CN12_58: (no net) -> unconnected-(U1B-PF3-PadCN12_58)
- U1 pad CN12_59: (no net) -> unconnected-(U1B-PF12-PadCN12_59)
- U1 pad CN12_6: (no net) -> unconnected-(U1B-PC5-PadCN12_6)
- U1 pad CN12_60: (no net) -> unconnected-(U1B-PF15-PadCN12_60)
- U1 pad CN12_61: (no net) -> unconnected-(U1B-PG14-PadCN12_61)
- U1 pad CN12_62: (no net) -> unconnected-(U1B-PF11-PadCN12_62)
- U1 pad CN12_63: (no net) -> Net-(U1B-GND_CN12-PadCN12_20)
- U1 pad CN12_64: (no net) -> unconnected-(U1B-PE0-PadCN12_64)
- U1 pad CN12_65: (no net) -> unconnected-(U1B-PD10-PadCN12_65)
- U1 pad CN12_66: (no net) -> unconnected-(U1B-PG8-PadCN12_66)
- U1 pad CN12_67: (no net) -> unconnected-(U1B-PG7-PadCN12_67)
- U1 pad CN12_68: (no net) -> unconnected-(U1B-PG5-PadCN12_68)
- U1 pad CN12_69: (no net) -> unconnected-(U1B-PG4-PadCN12_69)
- U1 pad CN12_7: (no net) -> unconnected-(U1B-VREFP-PadCN12_7)
- U1 pad CN12_70: (no net) -> unconnected-(U1B-PG6-PadCN12_70)
- U1 pad CN12_71: (no net) -> Net-(U1B-GND_CN12-PadCN12_20)
- U1 pad CN12_72: (no net) -> Net-(U1B-GND_CN12-PadCN12_20)
- U1 pad CN12_8: (no net) -> unconnected-(U1B-5V_USB_STLK-PadCN12_8)
- U1 pad CN12_9: (no net) -> Net-(U1B-GND_CN12-PadCN12_20)
- U1 pad CN7_1: (no net) -> unconnected-(U1E-D16/I2S_A_MCK-PadCN7_1)
- U1 pad CN7_10: (no net) -> unconnected-(U1E-D13/SPI_A_SCK-PadCN7_10)
- U1 pad CN7_11: (no net) -> unconnected-(U1E-D21/I2S_B_MCK-PadCN7_11)
- U1 pad CN7_12: (no net) -> unconnected-(U1E-D12/SPI_A_MISO-PadCN7_12)
- U1 pad CN7_13: (no net) -> unconnected-(U1E-D22/I2S_B_SD/SPI_B_MOSI-PadCN7_13)
- U1 pad CN7_14: (no net) -> AAM_FMC_D0
- U1 pad CN7_15: (no net) -> unconnected-(U1E-D23/I2S_B_CK/SPI_B_SCK-PadCN7_15)
- U1 pad CN7_16: (no net) -> AAM_FMC_D1
- U1 pad CN7_17: (no net) -> unconnected-(U1E-D24/SPI_B_NSS-PadCN7_17)
- U1 pad CN7_18: (no net) -> unconnected-(U1E-D9/TIMER_B_PWM2-PadCN7_18)
- U1 pad CN7_19: (no net) -> unconnected-(U1E-D25/SPI_B_MISO-PadCN7_19)
- U1 pad CN7_2: (no net) -> unconnected-(U1E-D15/I2C_A_SCL-PadCN7_2)
- U1 pad CN7_20: (no net) -> unconnected-(U1E-D8/IO-PadCN7_20)
- U1 pad CN7_3: (no net) -> unconnected-(U1E-D17/I2S_A_SD-PadCN7_3)
- U1 pad CN7_4: (no net) -> unconnected-(U1E-D14/I2C_A_SDA-PadCN7_4)
- U1 pad CN7_5: (no net) -> unconnected-(U1E-D18/I2S_A_CK-PadCN7_5)
- U1 pad CN7_6: (no net) -> unconnected-(U1E-VREFP_CN7-PadCN7_6)
- U1 pad CN7_7: (no net) -> unconnected-(U1E-D19/I2S_A_WS-PadCN7_7)
- U1 pad CN7_8: (no net) -> unconnected-(U1E-GND_CN7-PadCN7_8)
- U1 pad CN7_9: (no net) -> unconnected-(U1E-D20/I2S_B_WS-PadCN7_9)
- U1 pad CN8_1: (no net) -> unconnected-(U1C-NC_CN8-PadCN8_1)
- U1 pad CN8_10: (no net) -> unconnected-(U1C-D47/SDMMC_CK-PadCN8_10)
- U1 pad CN8_11: (no net) -> Net-(U1C-GND_CN8-PadCN8_11)
- U1 pad CN8_12: (no net) -> unconnected-(U1C-D48/SDMMC_CMD-PadCN8_12)
- U1 pad CN8_13: (no net) -> Net-(U1C-GND_CN8-PadCN8_11)
- U1 pad CN8_14: (no net) -> unconnected-(U1C-D49/IO-PadCN8_14)
- U1 pad CN8_15: (no net) -> unconnected-(U1C-VIN_CN8-PadCN8_15)
- U1 pad CN8_16: (no net) -> unconnected-(U1C-D50/IO-PadCN8_16)
- U1 pad CN8_2: (no net) -> unconnected-(U1C-D43/SDMMC_D0-PadCN8_2)
- U1 pad CN8_3: (no net) -> unconnected-(U1C-IOREF_CN8-PadCN8_3)
- U1 pad CN8_4: (no net) -> unconnected-(U1C-D44/SDMMC_D1/I2S_A_CKIN-PadCN8_4)
- U1 pad CN8_5: (no net) -> unconnected-(U1C-NRST_CN8-PadCN8_5)
- U1 pad CN8_6: (no net) -> unconnected-(U1C-D45/SDMMC_D2-PadCN8_6)
- U1 pad CN8_7: (no net) -> unconnected-(U1C-3V3_CN8-PadCN8_7)
- U1 pad CN8_8: (no net) -> unconnected-(U1C-D46/SDMMC_D3-PadCN8_8)
- U1 pad CN8_9: (no net) -> unconnected-(U1C-5V_CN8-PadCN8_9)
- U1 pad CN9_1: (no net) -> unconnected-(U1D-A0/ADC12_INP15-PadCN9_1)
- U1 pad CN9_10: (no net) -> unconnected-(U1D-D55/USART_B_CTS-PadCN9_10)
- U1 pad CN9_11: (no net) -> unconnected-(U1D-A5/ADC3_INP6/I2C1_SCL-PadCN9_11)
- U1 pad CN9_12: (no net) -> Net-(U1D-GND_CN9-PadCN9_12)
- U1 pad CN9_13: (no net) -> unconnected-(U1D-D72/COMP1_INP-PadCN9_13)
- U1 pad CN9_14: (no net) -> unconnected-(U1D-D56/SAI_A_MCLK-PadCN9_14)
- U1 pad CN9_15: (no net) -> unconnected-(U1D-D71/COMP2_INP-PadCN9_15)
- U1 pad CN9_16: (no net) -> unconnected-(U1D-D57/SAI_A_FS-PadCN9_16)
- U1 pad CN9_17: (no net) -> unconnected-(U1D-D70/I2C_B_SMBA-PadCN9_17)
- U1 pad CN9_18: (no net) -> unconnected-(U1D-D58/SAI_A_SCK-PadCN9_18)
- U1 pad CN9_19: (no net) -> unconnected-(U1D-D69/I2C_B_SCL-PadCN9_19)
- U1 pad CN9_2: (no net) -> unconnected-(U1D-D51/USART_B_SCLK-PadCN9_2)
- U1 pad CN9_20: (no net) -> unconnected-(U1D-D59/SAI_A_SD-PadCN9_20)
- U1 pad CN9_21: (no net) -> unconnected-(U1D-D68/I2C_B_SDA-PadCN9_21)
- U1 pad CN9_22: (no net) -> unconnected-(U1D-D60/SAI_B_SD-PadCN9_22)
- U1 pad CN9_23: (no net) -> Net-(U1D-GND_CN9-PadCN9_12)
- U1 pad CN9_24: (no net) -> unconnected-(U1D-D61/SAI_B_SCK-PadCN9_24)
- U1 pad CN9_25: (no net) -> AAM_FMC_D3
- U1 pad CN9_26: (no net) -> unconnected-(U1D-D62/SAI_B_MCLK-PadCN9_26)
- U1 pad CN9_27: (no net) -> AAM_FMC_D2
- U1 pad CN9_28: (no net) -> unconnected-(U1D-D63/SAI_B_FS-PadCN9_28)
- U1 pad CN9_29: (no net) -> unconnected-(U1D-D65/IO-PadCN9_29)
- U1 pad CN9_3: (no net) -> unconnected-(U1D-A1/ADC123_INP10-PadCN9_3)
- U1 pad CN9_30: (no net) -> unconnected-(U1D-D64/IO-PadCN9_30)
- U1 pad CN9_4: (no net) -> unconnected-(U1D-D52/USART_B_RX-PadCN9_4)
- U1 pad CN9_5: (no net) -> unconnected-(U1D-A2/ADC12_INP13-PadCN9_5)
- U1 pad CN9_6: (no net) -> AAM_FMC_NWE
- U1 pad CN9_7: (no net) -> unconnected-(U1D-A3/ADC12_INP5-PadCN9_7)
- U1 pad CN9_8: (no net) -> AAM_FMC_NOE
- U1 pad CN9_9: (no net) -> unconnected-(U1D-A4/ADC123_INP12/I2C1_SDA-PadCN9_9)
- U3 pad CN10_20: Net-(U3B-GND_S2-PadCN10_20) -> GND
- U3 pad CN10_8: unconnected-(U3B-U5V-PadCN10_8) -> 5V_UUM
- U3 pad CN10_9: Net-(U3B-GND_S2-PadCN10_20) -> GND
Routing:
- net TDM_I2C1_SCL: track 420.4 -> 0.00 mm, vias 6 -> 0
- net TDM_I2C1_SDA: track 410.4 -> 0.00 mm, vias 1 -> 0
- net TDM_VDD: track 362.0 -> 0.00 mm, vias 7 -> 0
- net TDM_DBG_RX: track 278.7 -> 0.00 mm, vias 1 -> 0
- net TDM_DBG_TX: track 278.0 -> 0.00 mm, vias 1 -> 0
- net 5V_TDM: track 154.4 -> 0.00 mm, vias 6 -> 0
- net TDM_LED_FAIL: track 112.8 -> 0.00 mm, vias 2 -> 0
- net TDM_LED_OK: track 95.8 -> 0.00 mm, vias 1 -> 0
- net Net-(U1A-GND_CN11-PadCN11_19): track 91.4 -> 0.00 mm
- net Net-(U2A-GND_CN11-PadCN11_19): track 88.9 -> 0.00 mm
- net GND: track 76.4 -> 0.00 mm, vias 31 -> 0
- net TDM_LED_WARN: track 74.2 -> 0.00 mm, vias 1 -> 0
- net Net-(U9B-PC7): track 50.8 -> 0.00 mm
- net Net-(J10-Pin_1): track 26.6 -> 0.00 mm
- net Net-(J11-Pin_1): track 23.7 -> 0.00 mm
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Other:
- board size 536 x 151 mm -> 375.2 x 151 mm
- board text added: "HDMI"
- board text added: "LED_FAIL"
- board text added: "LED_OK"
- board text added: "LED_PWR"
- board text added: "LED_WARN"
- board text added: "USB-C"

Commit message: display driver schematic piece
Parts:
- added J3: LCD_display, Connector_PinHeader_1.00mm:PinHeader_1x04_P1.00mm_Horizontal, F.Cu at (334.7, 194.9)
- added U17: NUCLEO-H753ZI, NUCLEO-H753ZI:MODULE_NUCLEO-H753ZI, F.Cu at (448.1, 126.5)
- added U18: HDSP-7503, Display_7Segment:HDSP-A151, F.Cu at (213.2, 82.5)
- added U19: HDSP-7503, Display_7Segment:HDSP-A151, F.Cu at (222.5, 82.5)
- U2: value NUCLEO-H753ZI -> HDSP-7503; footprint NUCLEO-H753ZI:MODULE_NUCLEO-H753ZI -> Display_7Segment:HDSP-A151
- moved U2 248.1 mm to (203.9, 82.5)
Connections:
- J1 pad 10: ACM_LED_WARN -> ACM_LED_FAIL
- J1 pad 11: ACM_LED_FAIL -> ACM_LED_OK
- J1 pad 12: ACM_LED_OK -> ACM_LED_WARN
- J1 pad 13: AAM_FMC_A10 -> AAM_FMC_CLK
- J1 pad 14: AAM_FMC_A11 -> unconnected-(J1-Pin_14-Pad14)
- J1 pad 15: AAM_FMC_A12 -> unconnected-(J1-Pin_15-Pad15)
- J1 pad 16: AAM_FMC_A13 -> unconnected-(J1-Pin_16-Pad16)
- J1 pad 17: AAM_FMC_A14 -> unconnected-(J1-Pin_17-Pad17)
- J1 pad 18: AAM_FMC_A15 -> unconnected-(J1-Pin_18-Pad18)
- J1 pad 19: unconnected-(J1-Pin_19-Pad19) -> AAM_FMC_NWE
- J1 pad 20: unconnected-(J1-Pin_20-Pad20) -> AAM_FMC_NOE
- J1 pad 21: unconnected-(J1-Pin_21-Pad21) -> AAM_FMC_NE
- J1 pad 22: unconnected-(J1-Pin_22-Pad22) -> AAM_FMC_NL
- J1 pad 23: unconnected-(J1-Pin_23-Pad23) -> AAM_FMC_NBL0
- J1 pad 24: unconnected-(J1-Pin_24-Pad24) -> AAM_FMC_NBL1
- J2 pad 1: AAM_FMC_NWE -> AAM_FMC_D0
- J2 pad 10: AAM_FMC_D6 -> AAM_FMC_D9
- J2 pad 11: AAM_FMC_D7 -> AAM_FMC_D10
- J2 pad 12: AAM_FMC_A0 -> AAM_FMC_D11
- J2 pad 13: AAM_FMC_A1 -> AAM_FMC_D12
- J2 pad 14: AAM_FMC_A2 -> AAM_FMC_D13
- J2 pad 15: AAM_FMC_A3 -> ACM_FMC_D14
- J2 pad 16: AAM_FMC_A4 -> ACM_FMC_D15
- J2 pad 19: AAM_FMC_A6 -> unconnected-(J2-Pin_19-Pad19)
- J2 pad 2: AAM_FMC_NOE -> AAM_FMC_D1
- J2 pad 20: AAM_FMC_A7 -> unconnected-(J2-Pin_20-Pad20)
- J2 pad 21: AAM_FMC_A8 -> unconnected-(J2-Pin_21-Pad21)
- J2 pad 22: AAM_FMC_A9 -> unconnected-(J2-Pin_22-Pad22)
- J2 pad 3: AAM_FMC_NCE -> AAM_FMC_D2
- J2 pad 4: AAM_FMC_D0 -> AAM_FMC_D3
- J2 pad 5: AAM_FMC_D1 -> AAM_FMC_D4
- J2 pad 6: AAM_FMC_D2 -> AAM_FMC_D5
- J2 pad 7: AAM_FMC_D3 -> AAM_FMC_D6
- J2 pad 8: AAM_FMC_D4 -> AAM_FMC_D7
- J2 pad 9: AAM_FMC_D5 -> AAM_FMC_D8
- J8 pad 10: ACM_LED_WARN -> ACM_LED_FAIL
- J8 pad 11: ACM_LED_FAIL -> ACM_LED_OK
- J8 pad 12: ACM_LED_OK -> ACM_LED_WARN
- J8 pad 13: AAM_FMC_A10 -> AAM_FMC_CLK
- J8 pad 14: AAM_FMC_A11 -> unconnected-(J1-Pin_14-Pad14)
- J8 pad 15: AAM_FMC_A12 -> unconnected-(J1-Pin_15-Pad15)
- J8 pad 16: AAM_FMC_A13 -> unconnected-(J1-Pin_16-Pad16)
- J8 pad 17: AAM_FMC_A14 -> unconnected-(J1-Pin_17-Pad17)
- J8 pad 18: AAM_FMC_A15 -> unconnected-(J1-Pin_18-Pad18)
- J8 pad 19: unconnected-(J8-Pin_19-Pad19) -> AAM_FMC_NWE
- J8 pad 20: unconnected-(J8-Pin_20-Pad20) -> AAM_FMC_NOE
- J8 pad 21: unconnected-(J8-Pin_21-Pad21) -> AAM_FMC_NE
- J8 pad 22: unconnected-(J8-Pin_22-Pad22) -> AAM_FMC_NL
- J8 pad 23: unconnected-(J8-Pin_23-Pad23) -> AAM_FMC_NBL0
- J8 pad 24: unconnected-(J8-Pin_24-Pad24) -> AAM_FMC_NBL1
- J9 pad 1: AAM_FMC_NWE -> AAM_FMC_D0
- J9 pad 10: AAM_FMC_D6 -> AAM_FMC_D9
- J9 pad 11: AAM_FMC_D7 -> AAM_FMC_D10
- J9 pad 12: AAM_FMC_A0 -> AAM_FMC_D11
- J9 pad 13: AAM_FMC_A1 -> AAM_FMC_D12
- J9 pad 14: AAM_FMC_A2 -> AAM_FMC_D13
- J9 pad 15: AAM_FMC_A3 -> ACM_FMC_D14
- J9 pad 16: AAM_FMC_A4 -> ACM_FMC_D15
- J9 pad 17: AAM_FMC_A5 -> unconnected-(J9-Pin_17-Pad17)
- J9 pad 19: AAM_FMC_A6 -> unconnected-(J2-Pin_19-Pad19)
- J9 pad 2: AAM_FMC_NOE -> AAM_FMC_D1
- J9 pad 20: AAM_FMC_A7 -> unconnected-(J2-Pin_20-Pad20)
- J9 pad 21: AAM_FMC_A8 -> unconnected-(J2-Pin_21-Pad21)
- J9 pad 22: AAM_FMC_A9 -> unconnected-(J2-Pin_22-Pad22)
- J9 pad 3: AAM_FMC_NCE -> AAM_FMC_D2
- J9 pad 4: AAM_FMC_D0 -> AAM_FMC_D3
- J9 pad 5: AAM_FMC_D1 -> AAM_FMC_D4
- J9 pad 6: AAM_FMC_D2 -> AAM_FMC_D5
- J9 pad 7: AAM_FMC_D3 -> AAM_FMC_D6
- J9 pad 8: AAM_FMC_D4 -> AAM_FMC_D7
- J9 pad 9: AAM_FMC_D5 -> AAM_FMC_D8
- U1 pad CN10_16: AAM_FMC_D4 -> unconnected-(U1F-D0/USART_A_RX-PadCN10_16)
- U1 pad CN10_18: AAM_FMC_D5 -> unconnected-(U1F-D42/TIMER_A_PWM1N-PadCN10_18)
- U1 pad CN10_20: AAM_FMC_D4 -> unconnected-(U1F-D41/TIMER_A_ETR-PadCN10_20)
- U1 pad CN10_24: AAM_FMC_D7 -> unconnected-(U1F-D40/TIMER_A_PWM2N-PadCN10_24)
- U1 pad CN10_4: AAM_FMC_D6 -> unconnected-(U1F-D6/TIMER_A_PWM1-PadCN10_4)
- U1 pad CN11_21: unconnected-(U1A-PB7-PadCN11_21) -> AAM_FMC_NL
- U1 pad CN11_39: unconnected-(U1A-PD4-PadCN11_39) -> AAM_FMC_NOE
- U1 pad CN11_40: unconnected-(U1A-PD3-PadCN11_40) -> AAM_FMC_CLK
- U1 pad CN11_41: unconnected-(U1A-PD5-PadCN11_41) -> AAM_FMC_NWE
- U1 pad CN11_55: unconnected-(U1A-PD1-PadCN11_55) -> AAM_FMC_D3
- U1 pad CN11_57: unconnected-(U1A-PD0-PadCN11_57) -> AAM_FMC_D2
- U1 pad CN11_61: unconnected-(U1A-PE1-PadCN11_61) -> AAM_FMC_NBL1
- U1 pad CN11_69: unconnected-(U1A-PD9-PadCN11_69) -> ACM_FMC_D14
- U1 pad CN12_10: unconnected-(U1B-PD8-PadCN12_10) -> AAM_FMC_D13
- U1 pad CN12_19: AAM_FMC_NCE -> AAM_FMC_NE
- U1 pad CN12_40: unconnected-(U1B-PE8-PadCN12_40) -> AAM_FMC_D5
- U1 pad CN12_44: unconnected-(U1B-PE7-PadCN12_44) -> AAM_FMC_D4
- U1 pad CN12_46: unconnected-(U1B-PD14-PadCN12_46) -> AAM_FMC_D0
- U1 pad CN12_47: unconnected-(U1B-PE10-PadCN12_47) -> AAM_FMC_D7
- U1 pad CN12_48: unconnected-(U1B-PD15-PadCN12_48) -> AAM_FMC_D1
- U1 pad CN12_49: unconnected-(U1B-PE12-PadCN12_49) -> AAM_FMC_D9
- U1 pad CN12_51: unconnected-(U1B-PE14-PadCN12_51) -> AAM_FMC_D11
- U1 pad CN12_52: unconnected-(U1B-PE9-PadCN12_52) -> AAM_FMC_D6
- U1 pad CN12_53: unconnected-(U1B-PE15-PadCN12_53) -> AAM_FMC_D12
- U1 pad CN12_55: unconnected-(U1B-PE13-PadCN12_55) -> AAM_FMC_D10
- U1 pad CN12_56: unconnected-(U1B-PE11-PadCN12_56) -> AAM_FMC_D8
- U1 pad CN12_64: unconnected-(U1B-PE0-PadCN12_64) -> AAM_FMC_NBL0
- U1 pad CN12_65: unconnected-(U1B-PD10-PadCN12_65) -> ACM_FMC_D15
- U1 pad CN7_14: AAM_FMC_D0 -> unconnected-(U1E-D11/SPI_A_MOSI/TIM_E_PWM1-PadCN7_14)
- U1 pad CN7_16: AAM_FMC_D1 -> unconnected-(U1E-D10/SPI_A_CS/TIM_B_PWM3-PadCN7_16)
- U1 pad CN9_25: AAM_FMC_D3 -> unconnected-(U1D-D67/CAN_RX-PadCN9_25)
- U1 pad CN9_27: AAM_FMC_D2 -> unconnected-(U1D-D66/CAN_TX-PadCN9_27)
- U1 pad CN9_6: AAM_FMC_NWE -> unconnected-(U1D-D53/USART_B_TX-PadCN9_6)
- U1 pad CN9_8: AAM_FMC_NOE -> unconnected-(U1D-D54/USART_B_RTS-PadCN9_8)
- U4 pad 10: unconnected-(U4-PA15-Pad10) -> Net-(U2-F)
- U4 pad 11: unconnected-(U4-PB3-Pad11) -> Net-(U2-E)
- U4 pad 12: unconnected-(U4-PB4-Pad12) -> Net-(U2-D)
- U4 pad 13: unconnected-(U4-PB5-Pad13) -> Net-(U2-C)
- U4 pad 14: unconnected-(U4-PB6-Pad14) -> Net-(U2-B)
- U4 pad 15: unconnected-(U4-PB7-Pad15) -> Net-(U2-A)
- U4 pad 16: unconnected-(U4-PB8-Pad16) -> Net-(U18-DP)
- U4 pad 17: unconnected-(U4-PB9-Pad17) -> Net-(U18-G)
- U4 pad 18: unconnected-(U4-5V-Pad18) -> 5V_7SDD
- U4 pad 23: unconnected-(U4-PC14-Pad23) -> Net-(U18-F)
- U4 pad 24: unconnected-(U4-PC15-Pad24) -> Net-(U18-E)
- U4 pad 25: unconnected-(U4-PA0-Pad25) -> Net-(U18-D)
- U4 pad 26: unconnected-(U4-PA1-Pad26) -> Net-(U18-C)
- U4 pad 27: unconnected-(U4-PA2-Pad27) -> Net-(U18-B)
- U4 pad 28: unconnected-(U4-PA3-Pad28) -> Net-(U18-A)
- U4 pad 29: unconnected-(U4-PA4-Pad29) -> Net-(U19-DP)
- U4 pad 30: unconnected-(U4-PA5-Pad30) -> Net-(U19-G)
- U4 pad 31: unconnected-(U4-PA6-Pad31) -> Net-(U19-F)
- U4 pad 32: unconnected-(U4-PA7-Pad32) -> Net-(U19-E)
- U4 pad 33: unconnected-(U4-PB0-Pad33) -> Net-(U19-D)
- U4 pad 34: unconnected-(U4-PB1-Pad34) -> Net-(U19-C)
- U4 pad 35: unconnected-(U4-PB10-Pad35) -> Net-(U19-B)
- U4 pad 36: unconnected-(U4-PB11-Pad36) -> Net-(U19-A)
- U4 pad 39: unconnected-(U4-GND-Pad39) -> GND
- U4 pad 8: unconnected-(U4-PA11-Pad8) -> Net-(U2-DP)
- U4 pad 9: unconnected-(U4-PA12-Pad9) -> Net-(U2-G)
Other:
- board text added: "DSM_DBG"
