File: schematic/signalmesh.kicad_pcb (KiCad board)
At the start: 4 copper layers, 387 x 151 mm, 137 parts, among them J1 FPGA I/O, J10 INA219_CONFIG, J11 INA219_CONFIG, J12 AAM_DBG, J13 DSM_DBG, J14 ACM_DBG, J15 INA219_CONFIG, J16 DSM_DBG, J17 LCD_display, J18 LCD_display, J19 AudioJack3, J2 FPGA I/O, J3 LCD_display, J4 TDM_DBG, J5 INA219_CONFIG, J6 INA219_CONFIG, J7 INA219_CONFIG, J8 FPGA I/O, J9 FPGA I/O, U1 NUCLEO-H753ZI, U10 INA219AxD, U11 INA219AxD, U12 INA219AxD, U13 INA219AxD, U14 W25Q128JVS, U15 AP2112K-3.3, U16 74HC4050D, U17 NUCLEO-H753ZI, U18 HDSP-7503, U19 HDSP-7503, U2 HDSP-7503, U20 INA219AxD, U21 74HC4050D, U22 AP2112K-3.3, U23 W25Q128JVS, U24 74HC4050D, U25 AP2112K-3.3, U26 W25Q128JVS, U27 MCP2551-I-P, U28 74LVC1G3157, U29 MCP2551-I-P, U3 NUCLEO-F303RE, U30 MCP2551-I-P, U31 MCP2551-I-P, U4 YAAJ_BluePill_Part_Like, U5 24LC256-I_SN, U6 BME280, U7 INA219AxD, U8 24LC256-I_SN, U9 NUCLEO-F446RE

Commit message: good progress. build from here. bit of autorouter. not too shitty
Parts:
- J13: value DSM_DBG -> UUM_DBG
- moved R1 52.0 mm to (203.8, 80.0)
- moved D19 50.2 mm to (211.8, 80.0), turned to 180 degrees
- moved J16 37.5 mm to (392.2, 53.9)
- moved J13 37.4 mm to (354.8, 53.8)
- moved U18 19.6 mm to (227.3, 78.2)
- moved U2 6.75 mm to (245.0, 78.2)
- moved U19 6.70 mm to (236.2, 78.2)
- moved U28 1.02 mm to (230.8, 102.5)
Connections:
- J1 pad 7: ACM_CMD_TX -> AAM_CMD_RX
- J1 pad 8: ACM_CMD_RX -> AAM_CMD_TX
- J13 pad 1: DSM_DBG_TX -> UUM_DBG_TX
- J13 pad 2: DSM_DBG_RX -> UUM_DBG_RX
- J8 pad 7: ACM_CMD_TX -> AAM_CMD_RX
- J8 pad 8: ACM_CMD_RX -> AAM_CMD_TX
- U1 pad CN11_1: unconnected-(U1A-PC10-PadCN11_1) -> AAM_CMD_TX
- U1 pad CN11_2: unconnected-(U1A-PC11-PadCN11_2) -> AAM_CMD_RX
- U1 pad CN12_3: UUM_CAN_RD -> AAM_CAN_RD
- U1 pad CN12_5: UUM_CAN_TD -> AAM_CAN_TD
- U17 pad CN12_3: UUM_CAN_RD -> DSM_CAN_RD
- U17 pad CN12_5: UUM_CAN_TD -> DSM_CAN_TD
- U24 pad 3: UUM_SPI1_CS -> UUM_SPI2_CS
- U3 pad CN10_21: unconnected-(U3B-PA9-PadCN10_21) -> UUM_SPI2_CS
Routing:
- net UUM_CAN_TD: track 532.0 -> 265.2 mm, vias 2 -> 1
- net UUM_DBG_RX: track 0.00 -> 227.4 mm, vias 0 -> 1
- net AAM_CAN_TD: track 0.00 -> 220.5 mm, vias 0 -> 1
- net UUM_DBG_TX: track 0.00 -> 217.6 mm, vias 0 -> 1
- net AAM_CAN_RD: track 0.00 -> 215.3 mm, vias 0 -> 1
- net UUM_CAN_RD: track 478.4 -> 288.3 mm, vias 4 -> 2
- net UUM_SPI2_CS: track 0.00 -> 128.8 mm, vias 0 -> 2
- net AAM_CMD_TX: track 0.00 -> 125.9 mm, vias 0 -> 1
- net AAM_CMD_RX: track 0.00 -> 122.3 mm, vias 0 -> 1
- net ACM_FMC_D15: track 214.1 -> 96.4 mm
- net DSM_CAN_TD: track 0.00 -> 107.4 mm, vias 0 -> 1
- net DSM_CAN_RD: track 0.00 -> 95.5 mm
- net DSM_DBG_RX: track 102.3 -> 63.3 mm
- net DSM_DBG_TX: track 100.7 -> 61.8 mm
- net VDD_ACM: track 181.8 -> 218.3 mm, vias 3 -> 0
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Other:
- board text added: "AUDIO OUT"
- board text added: "JLCJLCJLCJLC"
- board text removed: "Audio Out"

Commit message: i sort of like this. verifying one more time before printing
Routing:
- net AAM_FMC_D6: track 93.5 -> 83.9 mm
- net TDM_VDD: track 294.1 -> 290.4 mm
- net GND: track 195.7 -> 194.4 mm
- net UUM_SPI_SEL: track 108.3 -> 109.6 mm

Commit message: adding JLCPCB files
Parts:
- added 5V_TDM_TEST: TestPoint_Keystone_5019_Miniature, TestPoint:TestPoint_Keystone_5019_Miniature, F.Cu at (555.2, 147.8)
- added 5V_UUM: TestPoint_Keystone_5019_Miniature, TestPoint:TestPoint_Keystone_5019_Miniature, F.Cu at (470.5, 198.2)
- added AAM_DAC_L: TestPoint_Keystone_5019_Miniature, TestPoint:TestPoint_Keystone_5019_Miniature, F.Cu at (261.5, 77.5)
- added AAM_DAC_R: TestPoint_Keystone_5019_Miniature, TestPoint:TestPoint_Keystone_5019_Miniature, F.Cu at (269.2, 77.5)
- added ACM_VDD: TestPoint_Keystone_5019_Miniature, TestPoint:TestPoint_Keystone_5019_Miniature, F.Cu at (527.2, 198.0)
- added D28: LED_PWR, LED_SMD:LED_0603_1608Metric, F.Cu at (265.8, 92.8)
- added D29: LED_OK, LED_SMD:LED_0603_1608Metric, F.Cu at (265.8, 105.5)
- added D30: LED_FAIL, LED_SMD:LED_0603_1608Metric, F.Cu at (265.8, 101.2)
- added D31: LED_WARN, LED_SMD:LED_0603_1608Metric, F.Cu at (265.8, 96.8)
- added DSM_VDD: TestPoint_Keystone_5019_Miniature, TestPoint:TestPoint_Keystone_5019_Miniature, F.Cu at (384.8, 80.5)
- added GND: TestPoint_Keystone_5019_Miniature, TestPoint:TestPoint_Keystone_5019_Miniature, F.Cu at (453.5, 198.0)
- added R45: 300, Resistor_SMD:R_0805_2012Metric_Pad1.20x1.40mm_HandSolder, F.Cu at (258.2, 93.0)
- added R46: 300, Resistor_SMD:R_0805_2012Metric_Pad1.20x1.40mm_HandSolder, F.Cu at (258.2, 105.8)
- added R48: 300, Resistor_SMD:R_0805_2012Metric_Pad1.20x1.40mm_HandSolder, F.Cu at (258.2, 101.5)
- added R49: 300, Resistor_SMD:R_0805_2012Metric_Pad1.20x1.40mm_HandSolder, F.Cu at (258.2, 97.2)
- added TDM_I2C1_SCL: TestPoint_Keystone_5019_Miniature, TestPoint:TestPoint_Keystone_5019_Miniature, F.Cu at (492.0, 198.2)
- added TDM_I2C1_SDA: TestPoint_Keystone_5019_Miniature, TestPoint:TestPoint_Keystone_5019_Miniature, F.Cu at (500.5, 198.2)
- added VDD_UUM: TestPoint_Keystone_5019_Miniature, TestPoint:TestPoint_Keystone_5019_Miniature, F.Cu at (406.8, 198.0)
Connections:
- U1 pad CN12_34: unconnected-(U1B-PC4-PadCN12_34) -> AAM_LED_FAIL
- U1 pad CN12_4: unconnected-(U1B-PC6-PadCN12_4) -> AAM_LED_OK
- U1 pad CN12_6: unconnected-(U1B-PC5-PadCN12_6) -> AAM_LED_WARN
- U17 pad CN12_34: unconnected-(U17B-PC4-PadCN12_34) -> DSM_LED_FAIL
- U17 pad CN12_4: unconnected-(U17B-PC6-PadCN12_4) -> DSM_LED_OK
- U17 pad CN12_6: unconnected-(U17B-PC5-PadCN12_6) -> DSM_LED_WARN
- U3 pad CN7_35: unconnected-(U3A-PC2-PadCN7_35) -> UUM_LED_OK
- U3 pad CN7_36: unconnected-(U3A-PC1-PadCN7_36) -> UUM_LED_WARN
- U3 pad CN7_38: unconnected-(U3A-PC0-PadCN7_38) -> UUM_LED_FAIL
Routing:
- net UUM_LED_FAIL: track 0.00 -> 159.2 mm
- net DSM_LED_FAIL: track 0.00 -> 150.0 mm, vias 0 -> 2
- net UUM_LED_OK: track 0.00 -> 140.3 mm
- net UUM_LED_WARN: track 0.00 -> 133.3 mm, vias 0 -> 2
- net DSM_LED_WARN: track 0.00 -> 106.2 mm
- net DSM_LED_OK: track 0.00 -> 98.8 mm, vias 0 -> 1
- net AAM_LED_FAIL: track 0.00 -> 69.4 mm, vias 0 -> 2
- net AAM_LED_WARN: track 0.00 -> 25.7 mm
- net AAM_LED_OK: track 0.00 -> 17.0 mm
- net VDD_UUM: track 438.3 -> 451.8 mm, vias 6 -> 8
- net TDM_I2C1_SDA: track 342.5 -> 355.6 mm, vias 11 -> 13
- net 5V_UUM: track 339.8 -> 351.1 mm, vias 4 -> 6
- net GND: track 194.4 -> 204.8 mm, vias 79 -> 84
- net 5V_TDM: track 170.2 -> 180.4 mm
- net UUM_SPI2_CS: track 128.8 -> 118.9 mm
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