File: schematic/signalmesh_revert2.kicad_pcb (KiCad board)
At the start: 4 copper layers, 387 x 151 mm, 137 parts, among them J1 FPGA I/O, J10 INA219_CONFIG, J11 INA219_CONFIG, J12 AAM_DBG, J13 DSM_DBG, J14 ACM_DBG, J15 INA219_CONFIG, J16 DSM_DBG, J17 LCD_display, J18 LCD_display, J19 AudioJack3, J2 FPGA I/O, J3 LCD_display, J4 TDM_DBG, J5 INA219_CONFIG, J6 INA219_CONFIG, J7 INA219_CONFIG, J8 FPGA I/O, J9 FPGA I/O, U1 NUCLEO-H753ZI, U10 INA219AxD, U11 INA219AxD, U12 INA219AxD, U13 INA219AxD, U14 W25Q128JVS, U15 AP2112K-3.3, U16 74HC4050D, U17 NUCLEO-H753ZI, U18 HDSP-7503, U19 HDSP-7503, U2 HDSP-7503, U20 INA219AxD, U21 74HC4050D, U22 AP2112K-3.3, U23 W25Q128JVS, U24 74HC4050D, U25 AP2112K-3.3, U26 W25Q128JVS, U27 MCP2551-I-P, U28 74LVC1G3157, U29 MCP2551-I-P, U3 NUCLEO-F303RE, U30 MCP2551-I-P, U31 MCP2551-I-P, U4 YAAJ_BluePill_Part_Like, U5 24LC256-I_SN, U6 BME280, U7 INA219AxD, U8 24LC256-I_SN, U9 NUCLEO-F446RE

Commit message: ugh routing is a bit messy right now. need to go back to schematic and finish up wiring i forgot about primarily the UARTs for debugging on all boards and the cmd UART from AAM<->ACM
Parts:
- C1, C10, C2, C3, C4, C5, C6, C7, C8, C9: footprint Capacitor_SMD:C_0805_2012Metric -> Capacitor_SMD:C_0201_0603Metric
- D1, D10, D11, D12, D13, D14, D15, D16, D17, D18, D19, D2, D20, D21, D22, D23, D24, D25, D26, D27, D3, D4, D5, D6, D7, D8, D9: footprint LED_SMD:LED_0603_1608Metric -> LED_SMD:LED_Kingbright_KPBD-3224
- J17, J18, J3: footprint Connector_PinHeader_1.00mm:PinHeader_1x04_P1.00mm_Vertical_SMD_Pin1Left -> Connector_PinHeader_1.00mm:PinHeader_1x04_P1.00mm_Horizontal
Routing:
- net UUM_CAN_TD: track 532.0 -> 283.1 mm, vias 2 -> 1
- net UUM_CAN_RD: track 478.4 -> 274.3 mm, vias 4 -> 1
- net TDM_CAN_TD: track 118.0 -> 0.00 mm, vias 2 -> 0
- net TDM_CAN_RD: track 105.5 -> 0.00 mm, vias 2 -> 0
- net Net-(D11-A): track 0.00 -> 11.7 mm
- net Net-(D3-A): track 6.36 -> 11.6 mm, vias 0 -> 1
- net GND: track 191.3 -> 186.8 mm, vias 78 -> 75
- net Net-(D4-A): track 8.76 -> 13.1 mm, vias 0 -> 1
- net unconnected-(J2-Pin_22-Pad22): track 9.18 -> 13.6 mm
- net Net-(D1-A): track 6.55 -> 10.9 mm, vias 0 -> 1
- net Net-(D2-A): track 9.51 -> 11.6 mm, vias 0 -> 1
- net Net-(U21-4Y): track 19.3 -> 20.9 mm
- net Net-(D12-A): track 10.8 -> 12.2 mm
- net Net-(U14-~{CS}): track 20.3 -> 18.9 mm
- net 5V_TDM: track 175.6 -> 174.5 mm
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