File: schematic/v2/signalmesh.kicad_sch (KiCad schematic)
At the start: 104 parts, among them J10 INA219_CONFIG, J11 INA219_CONFIG, J13 UUM_DBG, J14 ACM_DBG, J15 INA219_CONFIG, J18 LCD_display, J4 TDM_DBG, J5 INA219_CONFIG, J6 INA219_CONFIG, J7 INA219_CONFIG, U10 INA219AxD, U11 INA219AxD, U12 INA219AxD, U13 INA219AxD, U14 W25Q128JVS, U15 AP2112K-3.3, U16 74HC4050D, U20 INA219AxD, U21 74HC4050D, U22 AP2112K-3.3, U23 W25Q128JVS, U24 74HC4050D, U25 AP2112K-3.3, U26 W25Q128JVS, U27 MCP2551-I-P, U28 74LVC1G3157, U29 MCP2551-I-P, U3 NUCLEO-F303RE, U30 MCP2551-I-P, U31 MCP2551-I-P, U5 24LC256-I_SN, U6 BME280, U7 INA219AxD, U8 24LC256-I_SN, U9 NUCLEO-F446RE

Commit message: moving AAM -> APM. creatint some abstraction like stuff
Parts:
- removed C1, C2, C3, C4, C5, C7: 0.1uf, Capacitor_SMD:C_0805_2012Metric, symbol Device:C_Small
- removed C6: 10uf, Capacitor_SMD:C_0805_2012Metric, symbol Device:C_Small
- removed D1: LED_OK, LED_SMD:LED_0603_1608Metric, symbol Device:LED
- removed D10, D20, D4, D5, D6, D7, D8, D9: LED_PWR, LED_SMD:LED_0603_1608Metric, symbol Device:LED
- removed D2: LED_FAIL, LED_SMD:LED_0603_1608Metric, symbol Device:LED
- removed D3: LED_WARN, LED_SMD:LED_0603_1608Metric, symbol Device:LED
- removed J10, J11, J15, J5, J6, J7: INA219_CONFIG, Connector_PinHeader_1.00mm:PinHeader_1x02_P1.00mm_Horizontal, symbol Connector_Generic:Conn_01x02
- removed J14: ACM_DBG, Connector_PinHeader_1.00mm:PinHeader_1x03_P1.00mm_Horizontal, symbol Connector_Generic:Conn_01x03
- removed J18: LCD_display, Connector_PinHeader_1.00mm:PinHeader_1x04_P1.00mm_Vertical_SMD_Pin1Left, symbol Connector_Generic:Conn_01x04
- removed J4: TDM_DBG, Connector_PinHeader_1.00mm:PinHeader_1x03_P1.00mm_Horizontal, symbol Connector_Generic:Conn_01x03
- removed R11, R12: 4.7k, Resistor_SMD:R_0805_2012Metric_Pad1.20x1.40mm_HandSolder, symbol Device:R
- removed R13, R14, R19, R20, R21, R22, R23, R24, R25, R26, R28, R3, R4: 10k, Resistor_SMD:R_0805_2012Metric_Pad1.20x1.40mm_HandSolder, symbol Device:R
- removed R15, R16, R17, R18, R2, R27, R29, R30, R31, R32, R33: 300, Resistor_SMD:R_0805_2012Metric_Pad1.20x1.40mm_HandSolder, symbol Device:R
- removed TH1: 10k, OptoDevice:R_LDR_4.9x4.2mm_P2.54mm_Vertical, symbol Device:Thermistor
- removed U10, U11, U12, U13, U20, U7: INA219AxD, Package_SO:SOIC-8_3.9x4.9mm_P1.27mm, symbol Sensor_Energy:INA219AxD
- removed U14: W25Q128JVS, Package_SO:SOIC-8_5.3x5.3mm_P1.27mm, symbol Memory_Flash:W25Q128JVS
- removed U15: AP2112K-3.3, Package_TO_SOT_SMD:SOT-23-5, symbol Regulator_Linear:AP2112K-3.3
- removed U16: 74HC4050D, 74HC4050D:SO16, symbol 74HC4050D:74HC4050D
- removed U5, U8: 24LC256-I_SN, 24LC256-I_SN:SOIC127P600X175-8N, symbol 24LC256-I_SN:24LC256-I_SN
- removed U6: BME280, Package_LGA:Bosch_LGA-8_2.5x2.5mm_P0.65mm_ClockwisePinNumbering, symbol Sensor:BME280
- removed U9: NUCLEO-F446RE, NUCLEO-F446RE:MODULE_NUCLEO-F446RE, symbol NUCLEO-F446RE:NUCLEO-F446RE
Other:
- added sheet TDM (TDM.kicad_sch)
- note removed: "APM <-> ACM FMC bus"
- note removed: "APM <-> ACM cmd ctrl"
- note removed: "INA219 7SDD"
- note removed: "INA219 ACM"
- note removed: "INA219 APM"
- note removed: "INA219 DSM"
- note removed: "INA219 TDM"
- note removed: "INA219 UUM"
- note removed: "Telemetry Debug Module"
- note removed: "W25Q128 ACM"
- moved on the sheet: R44, R47, U27, U29, U30, U31
