File: schematic/v2/ACM_debug.kicad_sch (KiCad schematic)
At the start: 16 parts, among them J12 USB_A, J14 ACM_DBG, U32 CH340G, Y1 Crystal

Commit message: no errors in the ERC!
Connections:
- net GND: now also C11.1
- no-connect marks 0 -> 9
Other:
- note added: "ACM Debug Port"
- note added: "UART debug messages avaiable via a USB port and a 3 pin jumper for TX, RX, and GND UART connections"
- moved on the sheet: C12
