File: schematic/v2/APM_debug.kicad_sch (KiCad schematic)
At the start: 16 parts, among them J16 APM_DBG, J20 USB_A, U33 CH340G, Y2 Crystal

Commit message: no errors in the ERC!
Parts:
- removed C14, C15, C16: 22pf, Capacitor_SMD:C_0805_2012Metric, symbol Device:C_Small
- removed D39: LED_PWR, LED_SMD:LED_0603_1608Metric, symbol Device:LED
- removed D40: TXD, LED_SMD:LED_0603_1608Metric, symbol Device:LED
- removed D41: RXD, LED_SMD:LED_0603_1608Metric, symbol Device:LED
- removed J16: APM_DBG, Connector_PinHeader_1.00mm:PinHeader_1x03_P1.00mm_Horizontal, symbol Connector_Generic:Conn_01x03
- removed J20: USB_A, Connector_USB:USB_A_CNCTech_1001-011-01101_Horizontal, symbol Connector:USB_A
- removed R57, R58, R59, R60: 300, Resistor_SMD:R_0805_2012Metric_Pad1.20x1.40mm_HandSolder, symbol Device:R
- removed R61: 1k5, Resistor_SMD:R_0805_2012Metric_Pad1.20x1.40mm_HandSolder, symbol Device:R
- removed U33: CH340G, Package_SO:SOIC-16_3.9x9.9mm_P1.27mm, symbol Interface_USB:CH340G
- removed Y2: Crystal, symbol Device:Crystal
- added C23, C24, C25: 22pf, Capacitor_SMD:C_0805_2012Metric, symbol Device:C_Small
- added D53: LED_PWR, LED_SMD:LED_0603_1608Metric, symbol Device:LED
- added D54: RXD, LED_SMD:LED_0603_1608Metric, symbol Device:LED
- added D55: TXD, LED_SMD:LED_0603_1608Metric, symbol Device:LED
- added J25: USB_A, Connector_USB:USB_A_CNCTech_1001-011-01101_Horizontal, symbol Connector:USB_A
- added J26: APM_DBG, Connector_PinHeader_1.00mm:PinHeader_1x03_P1.00mm_Horizontal, symbol Connector_Generic:Conn_01x03
- added R72, R79, R80, R82: 300, Resistor_SMD:R_0805_2012Metric_Pad1.20x1.40mm_HandSolder, symbol Device:R
- added R81: 1k5, Resistor_SMD:R_0805_2012Metric_Pad1.20x1.40mm_HandSolder, symbol Device:R
- added U19: CH340G, Package_SO:SOIC-16_3.9x9.9mm_P1.27mm, symbol Interface_USB:CH340G
- added Y5: Crystal, symbol Device:Crystal
Connections:
- net APM_DBG_RX: now also J26.2 (Pin_2), R80.1, R81.1, R82.1, U19.2 (TXD), U19.3 (RXD)
- net APM_DBG_TX: now also J26.1 (Pin_1), R81.2
- net APM_VDD: now also C25.2, J25.1 (VBUS), R72.2, R79.2, U19.16 (VCC)
- net GND: now also C23.2, C24.2, C25.1, D53.1 (K), D54.1 (K), D55.1 (K), J25.4 (GND), J26.3 (Pin_3), U19.1 (GND), Y5.1, Y5.2
- net at D38.2 (A): now also R72.1
- new net: D55.2 (A), R80.2
- new net: D54.2 (A), R82.2
- new net: C24.1, U19.7 (XI)
- new net: D53.2 (A), R79.1
- new net: J25.2 (D-), U19.6 (UD-)
- new net: J25.3 (D+), U19.5 (UD+)
- new net: C23.1, U19.8 (XO)
- no-connect marks 0 -> 9
Other:
- note added: "APM Debug Port"
- note added: "UART debug messages avaiable via a USB port and a 3 pin jumper for TX, RX, and GND UART connections"
