File: schematic/v2/TDM_debug.kicad_sch (KiCad schematic)
At the start: 16 parts, among them J23 USB_A, J4 TDM_DBG, U34 CH340G, Y3 Crystal

Commit message: no errors in the ERC!
Connections:
- net GND: now also C17.1
- no-connect marks 0 -> 8
Other:
- note added: "TDM Debug Port"
- note added: "UART debug messages avaiable via a USB port and a 3 pin jumper for TX, RX, and GND UART connections"
- moved on the sheet: C18, J4
