File: schematic/v2/signalmesh.kicad_pcb (KiCad board)
At the start: 4 copper layers, 387 x 151 mm, 188 parts, among them J1 FPGA I/O, J10 INA219_CONFIG, J11 INA219_CONFIG, J12 AAM_DBG, J13 UUM_DBG, J14 ACM_DBG, J15 INA219_CONFIG, J16 DSM_DBG, J17 LCD_display, J18 LCD_display, J19 AudioJack3, J2 FPGA I/O, J20 USB_A, J21 USB_A, J22 USB_A, J23 USB_A, J3 LCD_display, J4 TDM_DBG, J5 INA219_CONFIG, J6 INA219_CONFIG, J7 INA219_CONFIG, J8 FPGA I/O, J9 FPGA I/O, U1 NUCLEO-H753ZI, U10 INA219AxD, U11 INA219AxD, U12 INA219AxD, U13 INA219AxD, U14 W25Q128JVS, U15 AP2112K-3.3, U16 74HC4050D, U17 NUCLEO-H753ZI, U18 HDSP-7503, U19 HDSP-7503, U2 HDSP-7503, U20 INA219AxD, U21 74HC4050D, U22 AP2112K-3.3, U23 W25Q128JVS, U24 74HC4050D, U25 AP2112K-3.3, U26 W25Q128JVS, U27 MCP2551-I-P, U28 74LVC1G3157, U29 MCP2551-I-P, U3 NUCLEO-F303RE, U30 MCP2551-I-P, U31 MCP2551-I-P, U33 CH340G, U4 YAAJ_BluePill_Part_Like, U5 24LC256-I_SN, U6 BME280, U7 INA219AxD, U8 24LC256-I_SN, U9 NUCLEO-F446RE

Commit message: attempting new PCB layout
Parts:
- moved D19 3.55 mm to (208.2, 80.0)
Routing:
- net Net-(D19-A): track 6.26 -> 2.71 mm
Other:
- board text added: "signalmesh dev board v2.0 by Akiel Aries 2025"
- board text removed: "signalmesh dev board v1.0 by Akiel Aries 2025"
Changed lines of the file:
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@@
 	(footprint "LED_SMD:LED_0603_1608Metric"
 		(layer "F.Cu")
-		(at 211.8 80 180)
+		(at 208.25 80 180)
 		(descr "LED SMD 0603 (1608 Metric), square (rectangular) end terminal, IPC-7351 nominal, (Body size source: http://www.tortai-tech.com/upload/download/2011102023233369053.pdf), generated with kicad-footprint-generator")
 		(tags "LED")
 		(property "Reference" "D19"
-			(at 0 -1.43 0)
+			(at 0 -1.75 0)
 			(layer "F.SilkS")
 			(effects
@@
 		)
 		(fp_text user "1"
-			(at -1.6 -2.15 180)
+			(at -1.5 -2.15 180)
 			(unlocked yes)
 			(layer "F.SilkS")
@@
 		(tags "resistor handsolder")
 		(property "Reference" "R1"
-			(at 0 -1.65 0)
+			(at 0 -1.75 0)
 			(layer "F.SilkS")
 			(effects
@@
 	(gr_rect
 		(start 200.75 76.25)
-		(end 222.25 82.75)
+		(end 215.5 82.75)
 		(stroke
 			(width 0.2)
@@
 	)
 	(gr_text "PWR"
-		(at 215.55 80.75 0)
+		(at 210.5 80.75 0)
 		(layer "F.SilkS")
 		(effects
@@
 		)
 	)
-	(gr_text "signalmesh dev board v1.0\nby Akiel Aries 2025"
+	(gr_text "signalmesh dev board v2.0\nby Akiel Aries 2025"
 		(at 189.5 96.25 90)
 		(layer "F.SilkS")
@@
 	)
 	(segment
-		(start 211.012 80)
-		(end 204.75 80)
+		(start 207.4625 80)
+		(end 207.462 80)
 		(width 0.3)
 		(layer "F.Cu")
@@
 	)
 	(segment
-		(start 211.0125 80)
-		(end 211.012 80)
+		(start 207.4625 80)
+		(end 204.75 80)
 		(width 0.3)
 		(layer "F.Cu")
@@
 	)
 	(segment
-		(start 213.3 80)
-		(end 212.588 80)
+		(start 209.75 80)
+		(end 209.038 80)
 		(width 0.3)
 		(layer "F.Cu")
@@
 	)
 	(segment
-		(start 213.8 79.5)
-		(end 213.3 80)
+		(start 210.25 79.5)
+		(end 209.75 80)
 		(width 0.3)
 		(layer "F.Cu")
@@
 	)
 	(via
-		(at 213.8 79.5)
+		(at 210.25 79.5)
 		(size 0.6)
 		(drill 0.3)
@@
 	)
 	(segment
-		(start 524.75 189.5)
-		(end 518.75 195.5)
+		(start 524.75 165.75)
+		(end 524.75 189.5)
 		(width 0.5)
 		(layer "F.Cu")
@@
 	)
 	(segment
-		(start 542.1 165.3)
-		(end 525.2 165.3)
+		(start 397.21 167.48)
+		(end 396.5632 167.48)
 		(width 0.5)
 		(layer "F.Cu")
@@
 	)
 	(segment
-		(start 524.75 165.75)
-		(end 524.75 189.5)
+		(start 543.1 161.5)
+		(end 543.1 164.3)
 		(width 0.5)
 		(layer "F.Cu")
@@
 	)
 	(segment
-		(start 397.21 167.48)
-		(end 396.5632 167.48)
+		(start 543.85 160.75)
+		(end 543.1 161.5)
 		(width 0.5)
 		(layer "F.Cu")
@@
 	)
 	(segment
-		(start 525.2 165.3)
-		(end 524.75 165.75)
+		(start 542.1 165.3)
+		(end 525.2 165.3)
 		(width 0.5)
 		(layer "F.Cu")
@@
 	)
 	(segment
+		(start 524.75 189.5)
+		(end 518.75 195.5)
+		(width 0.5)
+		(layer "F.Cu")
+		(net 206)
+	)
+	(segment
+		(start 525.2 165.3)
+		(end 524.75 165.75)
+		(width 0.5)
+		(layer "F.Cu")
+		(net 206)
+	)
+	(segment
 		(start 544.849 161.749)
 		(end 543.85 160.75)
@@
 	)
 	(segment
-		(start 543.1 161.5)
-		(end 543.1 164.3)
+		(start 543.1 164.3)
+		(end 542.1 165.3)
 		(width 0.5)
 		(layer "F.Cu")
@@
 		(width 0.5)
 		(layer "F.Cu")
-		(net 206)
-	)
-	(segment
-		(start 543.85 160.75)
-		(end 543.1 161.5)
-		(width 0.5)
-		(layer "F.Cu")
-		(net 206)
-	)
-	(segment
-		(start 543.1 164.3)
-		(end 542.1 165.3)
-		(width 0.5)
-		(layer "F.Cu")
