File: schematic/v2/signalmesh.kicad_pcb (KiCad board)
At the start: 4 copper layers, 387 x 151 mm, 245 parts, among them J1 FPGA I/O, J10 INA219_CONFIG, J11 INA219_CONFIG, J12 AUDIO_OUT, J15 INA219_CONFIG, J18 LCD_display, J2 FPGA I/O, J21 USB_A, J22 USB_A, J25 USB_A, J26 UART_DEBUG, J27 USB_A, J28 UART_DEBUG, J29 USB_A, J3 LCD_display, J30 UART_DEBUG, J31 USB_A, J32 UART_DEBUG, J33 USB_A, J34 UART_DEBUG, J4 LCD_display, J5 INA219_CONFIG, J6 INA219_CONFIG, J7 INA219_CONFIG, J8 FPGA I/O, J9 FPGA I/O, U1 NUCLEO-H753ZI, U10 INA219AxD, U11 INA219AxD, U12 INA219AxD, U13 INA219AxD, U14 W25Q128JVS, U15 AP2112K-3.3, U16 74HC4050D, U17 NUCLEO-H753ZI, U18 SM420561N, U19 CH340G, U2 SM420561N, U20 INA219AxD, U21 74HC4050D, U22 AP2112K-3.3, U23 W25Q128JVS, U24 74HC4050D, U25 AP2112K-3.3, U26 W25Q128JVS, U27 MCP2551-I-P, U28 74LVC1G3157, U29 MCP2551-I-P, U3 NUCLEO-F303RE, U30 MCP2551-I-P, U31 MCP2551-I-P, U36 SM420561N, U37 CH340G, U38 CH340G, U39 CH340G, U4 YAAJ_BluePill_Part_Like, U40 CH340G, U5 24LC256-I_SN, U6 BME280, U7 INA219AxD, U8 24LC256-I_SN, U9 NUCLEO-F446RE, Y2 12MHz, Y5 12MHz, Y7 12MHz, Y8 12MHz, Y9 12MHz

Commit message: routed with no errors. could probably do some more verification before sending the initial order of the v2 revamp then start designing out the AFFM module
Routing:
- net /TDM/TDM_I2C1_SCL: track 0.00 -> 565.3 mm, vias 0 -> 6
- net /TDM/TDM_I2C1_SDA: track 0.00 -> 559.8 mm, vias 0 -> 9
- net TDM_VDD: track 159.8 -> 688.8 mm, vias 2 -> 16
- net APM_VDD: track 40.8 -> 523.9 mm, vias 2 -> 6
- net UUM_VDD: track 36.9 -> 465.8 mm, vias 2 -> 9
- net 5V_7SDD: track 0.00 -> 397.0 mm, vias 0 -> 3
- net /UUM_CAN_RD: track 0.00 -> 344.2 mm, vias 0 -> 1
- net /UUM_CAN_TD: track 0.00 -> 324.6 mm, vias 0 -> 1
- net /DAC_L: track 9.14 -> 307.0 mm, vias 0 -> 1
- net DSM_VDD: track 40.8 -> 332.6 mm, vias 2 -> 9
- net Net-(U9A-PA4): track 0.00 -> 265.8 mm
- net /DAC_R: track 9.07 -> 246.7 mm, vias 0 -> 1
- net /APM_CAN_RD: track 0.00 -> 229.4 mm, vias 0 -> 1
- net /APM_CAN_TD: track 0.00 -> 228.7 mm, vias 0 -> 1
- net Net-(U9A-PB0): track 0.00 -> 185.2 mm
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Other:
- board size 387 x 151 mm -> 515 x 152.4 mm
- board text added: "Analog Filter & FX Module AFFM"

Commit message: routed. saving the extra board in the same pcb file for when I want to creat the filter and fx module
Parts:
- moved OSHW 46.6 mm to (606.0, 158.0)
- moved R75 18.0 mm to (505.8, 117.0), turned to 180 degrees
- moved U18 6.54 mm to (216.4, 140.0)
- moved U2 6.54 mm to (202.5, 140.0)
- moved U36 6.54 mm to (188.5, 140.0)
Routing:
- net /ACM_DBG_RX: track 169.5 -> 137.1 mm
- net /ACM_DBG_TX: track 167.0 -> 138.2 mm
- net /UUM/UUM_SPI1_MISO: track 79.1 -> 63.1 mm, vias 3 -> 2
- net Net-(U30-Rs): track 13.9 -> 2.97 mm
- net /UUM/UUM_SPI_SEL: track 103.0 -> 95.7 mm, vias 2 -> 1
- net APM_VDD: track 523.9 -> 516.8 mm, vias 6 -> 7
- net /FMC_D6: track 135.0 -> 128.2 mm
- net Net-(U18-A): track 44.8 -> 51.4 mm
- net Net-(U36-E): track 27.7 -> 34.2 mm
- net Net-(U36-A): track 36.6 -> 43.2 mm
- net Net-(U36-D): track 23.7 -> 30.2 mm
- net Net-(U2-E): track 24.5 -> 31.0 mm
- net Net-(U2-DP): track 18.4 -> 25.0 mm
- net Net-(U2-D): track 25.2 -> 31.8 mm
- net Net-(U2-C): track 25.5 -> 32.0 mm
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Other:
- board size 515 x 152.4 mm -> 468.6 x 152.4 mm

Commit message: attempting v2 spinout with jlcpcb
Parts:
- moved R54 5.30 mm to (451.0, 86.0)
- moved R53 4.81 mm to (536.0, 57.0)
- moved R75 3.01 mm to (505.5, 114.0)
- moved TH2 2.49 mm to (309.8, 80.7)
- moved R57 1.98 mm to (242.6, 59.8)
- moved R74 1.16 mm to (489.4, 116.4)
Routing:
- net /ACM/ACM_SPI_MOSI: track 136.9 -> 117.1 mm
- net TDM_VDD: track 688.5 -> 682.0 mm, vias 16 -> 15
- net Net-(U9A-PC1/PB9): track 57.8 -> 62.8 mm
- net Net-(U9A-PC0/PB8): track 50.0 -> 53.3 mm
- net Net-(U9A-PB0): track 185.2 -> 187.6 mm
- net Net-(U9A-PA4): track 265.8 -> 267.9 mm
- net GND: track 283.8 -> 285.8 mm
- net Net-(U29-Rs): track 13.7 -> 15.3 mm
- net Net-(U30-Rs): track 2.97 -> 4.45 mm
- net Net-(U14-DI/IO_{0}): track 12.8 -> 13.4 mm
Other:
- board size 468.6 x 152.4 mm -> 387.9 x 152.3 mm
- board text removed: "Analog Filter & FX Module AFFM"
