File: schematic/v2/APM.kicad_sch (KiCad schematic)
At the start: 0 parts

Commit message: moving AAM -> APM. creatint some abstraction like stuff
Parts:
- added D15: LED_PWR, LED_SMD:LED_0603_1608Metric, symbol Device:LED
- added D16: LED_OK, LED_SMD:LED_0603_1608Metric, symbol Device:LED
- added D17: LED_FAIL, LED_SMD:LED_0603_1608Metric, symbol Device:LED
- added D18: LED_WARN, LED_SMD:LED_0603_1608Metric, symbol Device:LED
- added J19: AudioJack3, Connector_Audio:Jack_3.5mm_CUI_SJ-3523-SMT_Horizontal, symbol Connector_Audio:AudioJack3
- added J3: LCD_display, Connector_PinHeader_1.00mm:PinHeader_1x04_P1.00mm_Vertical_SMD_Pin1Left, symbol Connector_Generic:Conn_01x04
- added R38, R39, R40, R41: 300, Resistor_SMD:R_0805_2012Metric_Pad1.20x1.40mm_HandSolder, symbol Device:R
- added U1: NUCLEO-H753ZI, NUCLEO-H753ZI:MODULE_NUCLEO-H753ZI, symbol NUCLEO-H753ZI:NUCLEO-H753ZI
Connections:
- new net: D18.2 (A), R41.1
- new net: D15.2 (A), R38.1
- new net: U1.CN9_12 (GND_CN9), U1.CN9_23 (GND_CN9)
- new net: U1.CN11_10 (NC), U1.CN11_26 (NC), U1.CN11_67 (NC)
- new net: D16.2 (A), R39.1
- new net: D17.2 (A), R40.1
- new net: U1.CN10_17 (GND_CN10), U1.CN10_22 (GND_CN10), U1.CN10_27 (GND_CN10), U1.CN10_5 (GND_CN10)
- new net: U1.CN12_20 (GND_CN12), U1.CN12_39 (GND_CN12), U1.CN12_54 (GND_CN12), U1.CN12_63 (GND_CN12), U1.CN12_71 (GND_CN12), U1.CN12_72 (GND_CN12), U1.CN12_9 (GND_CN12)
- new net: U1.CN8_11 (GND_CN8), U1.CN8_13 (GND_CN8)
- new net 5V_APM: U1.CN11_18 (5V)
- new net APM_CAN_RD: U1.CN12_3 (PB8)
- new net APM_CAN_TD: U1.CN12_5 (PB9)
- new net APM_CMD_RX: U1.CN11_2 (PC11)
- new net APM_CMD_TX: U1.CN11_1 (PC10)
- new net APM_DAC_L: J19.T, U1.CN12_11 (PA5)
- new net APM_DAC_R: J19.R, U1.CN11_32 (PA4)
- new net APM_DBG_RX: U1.CN11_4 (PD2)
- new net APM_DBG_TX: U1.CN11_3 (PC12)
- new net APM_I2C1_SCL: J3.3 (Pin_3), U1.CN11_51 (PF1)
- new net APM_I2C1_SDA: J3.2 (Pin_2), U1.CN11_53 (PF0)
- new net APM_INTRPT_RX: U1.CN11_47 (PE3)
- new net APM_INTRPT_TX: U1.CN11_62 (PE6)
- new net APM_LED_FAIL: R41.2, U1.CN12_34 (PC4)
- new net APM_LED_OK: R39.2, U1.CN12_4 (PC6)
- new net APM_LED_WARN: R40.2, U1.CN12_6 (PC5)
- new net APM_USB_D+: U1.CN12_14 (PA11)
- new net APM_USB_D-: U1.CN12_12 (PA12)
- new net APM_VDD: J3.1 (Pin_1), R38.2
- new net GND: D15.1 (K), D16.1 (K), D17.1 (K), D18.1 (K), J19.S, J3.4 (Pin_4), U1.CN11_19 (GND_CN11), U1.CN11_20 (GND_CN11), U1.CN11_22 (GND_CN11), U1.CN11_49 (GND_CN11), U1.CN11_60 (GND_CN11), U1.CN11_71 (GND_CN11), U1.CN11_72 (GND_CN11), U1.CN11_8 (GND_CN11)
Other:
- added sheet 7SDD (7SDD.kicad_sch)
- added sheet APM_debug (APM_debug.kicad_sch)
- added sheet APM_midi (APM_midi.kicad_sch)
- note added: "STM32H755 NUCLEO"

Commit message: no errors in the ERC!
Parts:
- removed unit 4 of U1
- removed unit 5 of U1
- removed unit 6 of U1
- removed unit 3 of U1
Connections:
- net 7SDD_CMD_RX: now also U1.CN11_63 (PG9)
- net 7SDD_CMD_TX: now also U1.CN12_61 (PG14)
- no-connect marks 0 -> 11

Commit message: time to start routing?
Parts:
- removed J3: LCD_display, Connector_PinHeader_1.00mm:PinHeader_1x04_P1.00mm_Vertical_SMD_Pin1Left, symbol Connector_Generic:Conn_01x04
- added J4: LCD_display, Connector_PinHeader_1.00mm:PinHeader_1x04_P1.00mm_Horizontal, symbol Connector_Generic:Conn_01x04
Connections:
- net APM_VDD is gone; now on net 5V_APM: R38.2
- net 5V_APM: now also J4.1 (Pin_1)
- net APM_I2C1_SCL: now also J4.3 (Pin_3)
- net APM_I2C1_SDA: now also J4.2 (Pin_2)
- net GND: now also J4.4 (Pin_4)
Other:
- removed sheet APM_debug
Changed lines of the file:
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@@
 	(wire
 		(pts
-			(xy 45.72 57.15) (xy 59.69 57.15)
+			(xy 127 49.53) (xy 129.54 49.53)
 		)
 		(stroke
@@
 	(wire
 		(pts
-			(xy 76.2 110.49) (xy 88.9 110.49)
+			(xy 45.72 57.15) (xy 59.69 57.15)
 		)
 		(stroke
@@
 	(wire
 		(pts
-			(xy 45.72 76.2) (xy 58.42 76.2)
-		)
-		(stroke
-			(width 0)
-			(type default)
-		)
-	)
-	(wire
-		(pts
-			(xy 76.2 128.27) (xy 88.9 128.27)
-		)
-		(stroke
-			(width 0)
-			(type default)
-		)
-	)
-	(wire
-		(pts
 			(xy 124.46 148.59) (xy 127 148.59)
 		)
@@
 	(wire
 		(pts
-			(xy 45.72 80.01) (xy 58.42 80.01)
-		)
-		(stroke
-			(width 0)
-			(type default)
-		)
-	)
-	(wire
-		(pts
 			(xy 171.45 176.53) (xy 185.42 176.53)
 		)
@@
 		)
 	)
-	(label "APM_DBG_TX"
-		(at 76.2 110.49 0)
-		(effects
-			(font
-				(size 1.27 1.27)
-			)
-			(justify left bottom)
-		)
-	)
 	(label "APM_USB_D-"
 		(at 143.51 77.47 0)
@@
 		)
 	)
-	(label "APM_DBG_TX"
-		(at 58.42 80.01 180)
-		(effects
-			(font
-				(size 1.27 1.27)
-			)
-			(justify right bottom)
-		)
-	)
 	(label "7SDD_CMD_TX"
 		(at 59.69 60.96 180)
@@
 		)
 	)
-	(label "APM_DBG_RX"
-		(at 58.42 76.2 180)
-		(effects
-			(font
-				(size 1.27 1.27)
-			)
-			(justify right bottom)
-		)
-	)
 	(label "APM_I2C1_SDA"
 		(at 139.7 87.63 180)
@@
 		)
 	)
-	(label "APM_DBG_RX"
-		(at 76.2 128.27 0)
-		(effects
-			(font
-				(size 1.27 1.27)
-			)
-			(justify left bottom)
-		)
-	)
 	(label "APM_DAC_L"
 		(at 57.15 172.72 180)
@@
 		)
 	)
+	(hierarchical_label "APM_DBG_TX"
+		(shape output)
+		(at 88.9 110.49 180)
+		(effects
+			(font
+				(size 1.27 1.27)
+			)
+			(justify right)
+		)
+	)
 	(hierarchical_label "APM_CMD_RX"
 		(shape input)
@@
 		)
 	)
+	(hierarchical_label "APM_DBG_RX"
+		(shape input)
+		(at 88.9 128.27 180)
+		(effects
+			(font
+				(size 1.27 1.27)
+			)
+			(justify right)
+		)
+	)
 	(hierarchical_label "APM_CMD_TX"
 		(shape output)
@@
 		)
 	)
+	(hierarchical_label "APM_VDD"
+		(shape output)
+		(at 129.54 49.53 0)
+		(effects
+			(font
+				(size 1.27 1.27)
+			)
+			(justify left)
+		)
+	)
 	(hierarchical_label "APM_INTRPT_TX"
 		(shape output)
@@
 	)
 	(symbol
+		(lib_id "Connector_Generic:Conn_01x04")
+		(at 97.79 170.18 0)
+		(unit 1)
+		(exclude_from_sim no)
+		(in_bom yes)
+		(on_board yes)
+		(dnp no)
+		(fields_autoplaced yes)
+		(property "Reference" "J4"
+			(at 100.33 170.1799 0)
+			(effects
+				(font
+					(size 1.27 1.27)
+				)
+				(justify left)
+			)
+		)
+		(property "Value" "LCD_display"
+			(at 100.33 172.7199 0)
+			(effects
+				(font
+					(size 1.27 1.27)
+				)
+				(justify left)
+			)
+		)
+		(property "Footprint" "Connector_PinHeader_1.00mm:PinHeader_1x04_P1.00mm_Horizontal"
+			(at 97.79 170.18 0)
+			(effects
+				(font
+					(size 1.27 1.27)
+				)
+				(hide yes)
+			)
+		)
+		(property "Datasheet" "~"
+			(at 97.79 170.18 0)
+			(effects
+				(font
+					(size 1.27 1.27)
+				)
+				(hide yes)
+			)
+		)
+		(property "Description" "Generic connector, single row, 01x04, script generated (kicad-library-utils/schlib/autogen/connector/)"
+			(at 97.79 170.18 0)
+			(effects
+				(font
+					(size 1.27 1.27)
+				)
+				(hide yes)
+			)
+		)
+		(pin "3"
+		)
+		(pin "4"
+		)
+		(pin "2"
+		)
+		(pin "1"
+		)
+		(instances
+			(project "signalmesh"
+				(path "/fe7b15e9-f0ed-4338-9f03-dd7651dace13/0125ec8c-bf97-4530-be23-1f3b075b267b"
+					(reference "J4")
+					(unit 1)
+				)
+			)
+		)
+	)
+	(symbol
 		(lib_id "power:GND")
 		(at 161.29 160.02 0)
@@
 	)
 	(symbol
-		(lib_id "Connector_Generic:Conn_01x04")
-		(at 97.79 170.18 0)
-		(unit 1)
-		(exclude_from_sim no)
-		(in_bom yes)
-		(on_board yes)
-		(dnp no)
-		(fields_autoplaced yes)
-		(property "Reference" "J3"
-			(at 100.33 170.1799 0)
-			(effects
-				(font
-					(size 1.27 1.27)
-				)
-				(justify left)
-			)
-		)
-		(property "Value" "LCD_display"
-			(at 100.33 172.7199 0)
-			(effects
-				(font
-					(size 1.27 1.27)
-				)
-				(justify left)
-			)
-		)
-		(property "Footprint" "Connector_PinHeader_1.00mm:PinHeader_1x04_P1.00mm_Vertical_SMD_Pin1Left"
-			(at 97.79 170.18 0)
-			(effects
-				(font
-					(size 1.27 1.27)
-				)
-				(hide yes)
-			)
-		)
-		(property "Datasheet" "~"
-			(at 97.79 170.18 0)
-			(effects
-				(font
-					(size 1.27 1.27)
-				)
-				(hide yes)
-			)
-		)
-		(property "Description" "Generic connector, single row, 01x04, script generated (kicad-library-utils/schlib/autogen/connector/)"
-			(at 97.79 170.18 0)
-			(effects
-				(font
-					(size 1.27 1.27)
-				)
-				(hide yes)
-			)
-		)
-		(pin "3"
-		)
-		(pin "4"
-		)
-		(pin "2"
-		)
-		(pin "1"
-		)
-		(instances
-			(project "signalmesh"
-				(path "/fe7b15e9-f0ed-4338-9f03-dd7651dace13/0125ec8c-bf97-4530-be23-1f3b075b267b"
-					(reference "J3")
-					(unit 1)
-				)
-			)
-		)
-	)
-	(symbol
 		(lib_id "power:GND")
 		(at 127 148.59 0)
@@
 				)
 			)
-		)
-	)
-	(sheet
-		(at 30.48 72.39)
-		(size 15.24 11.43)
-		(exclude_from_sim no)
-		(in_bom yes)
-		(on_board yes)
-		(dnp no)
-		(fields_autoplaced yes)
-		(stroke
-			(width 0.1524)
-			(type solid)
-		)
-		(fill
-			(color 0 0 0 0.0000)
-		)
-		(property "Sheetname" "APM_debug"
-			(at 30.48 71.6784 0)
-			(effects
-				(font
-					(size 1.27 1.27)
-				)
-				(justify left bottom)
-			)
-		)
-		(property "Sheetfile" "APM_debug.kicad_sch"
-			(at 30.48 84.4046 0)
-			(effects
-				(font
-					(size 1.27 1.27)
-				)
-				(justify left top)
-			)
-		)
-		(pin "APM_DBG_TX" output
-			(at 45.72 76.2 0)
-			(effects
-				(font
-					(size 1.27 1.27)
-				)
-				(justify right)
-			)
-		)
-		(pin "APM_DBG_RX" input
-			(at 45.72 80.01 0)
-			(effects
-				(font
-					(size 1.27 1.27)
-				)
-				(justify right)
-			)
-		)
-		(instances
-			(project "signalmesh"
-				(path "/fe7b15e9-f0ed-4338-9f03-dd7651dace13/0125ec8c-bf97-4530-be23-1f3b075b267b"
-					(page "6")
-				)
-			)
