File: schematic/v2/DSM.kicad_sch (KiCad schematic)
At the start: 10 parts, among them J17 LCD_display, U17 NUCLEO-H753ZI

Commit message: attempting new PCB layout
Connections:
- net GND: no longer U17.CN12_20 (GND_CN12), U17.CN12_39 (GND_CN12), U17.CN12_54 (GND_CN12), U17.CN12_63 (GND_CN12), U17.CN12_71 (GND_CN12), U17.CN12_72 (GND_CN12), U17.CN12_9 (GND_CN12)
- new net: U17.CN12_20 (GND_CN12), U17.CN12_39 (GND_CN12), U17.CN12_54 (GND_CN12), U17.CN12_63 (GND_CN12), U17.CN12_71 (GND_CN12), U17.CN12_72 (GND_CN12), U17.CN12_9 (GND_CN12)
- no-connect marks 10 -> 11
Changed lines of the file:
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@@
+	)
+	(no_connect
+		(at 212.09 201.93)
 	)
 	(no_connect
@@
 		(pts
 			(xy 82.55 133.35) (xy 68.58 133.35)
-		)
-		(stroke
-			(width 0)
-			(type default)
-		)
-	)
-	(wire
-		(pts
-			(xy 215.9 201.93) (xy 212.09 201.93)
 		)
 		(stroke
@@
 					(unit 1)
 				)
-			)
-		)
-	)
-	(symbol
-		(lib_id "power:GND")
-		(at 215.9 201.93 0)
-		(unit 1)
-		(exclude_from_sim no)
-		(in_bom yes)
-		(on_board yes)
-		(dnp no)
-		(fields_autoplaced yes)
-		(property "Reference" "#PWR0179"
-			(at 215.9 208.28 0)
-			(effects
-				(font
-					(size 1.27 1.27)
-				)
-				(hide yes)
-			)
-		)
-		(property "Value" "GND"
-			(at 218.44 203.1999 0)
-			(effects
-				(font
-					(size 1.27 1.27)
-				)
-				(justify left)
-			)
-		)
-		(property "Footprint" ""
-			(at 215.9 201.93 0)
-			(effects
-				(font
-					(size 1.27 1.27)
-				)
-				(hide yes)
-			)
-		)
-		(property "Datasheet" ""
-			(at 215.9 201.93 0)
-			(effects
-				(font
-					(size 1.27 1.27)
-				)
-				(hide yes)
-			)
-		)
-		(property "Description" "Power symbol creates a global label with name \"GND\" , ground"
-			(at 215.9 201.93 0)
-			(effects
-				(font
-					(size 1.27 1.27)
-				)
-				(hide yes)
-			)
-		)
-		(pin "1"
-		)
-		(instances
-			(project "signalmesh"
-				(path "/fe7b15e9-f0ed-4338-9f03-dd7651dace13/4391c51f-6ab5-4b63-a6de-56382e56f1df"
-					(reference "#PWR0179")
-					(unit 1)
-				)

Commit message: time to start routing?
Parts:
- removed J17: LCD_display, Connector_PinHeader_1.00mm:PinHeader_1x04_P1.00mm_Vertical_SMD_Pin1Left, symbol Connector_Generic:Conn_01x04
- added J3: LCD_display, Connector_PinHeader_1.00mm:PinHeader_1x04_P1.00mm_Horizontal, symbol Connector_Generic:Conn_01x04
Connections:
- net DSM_VDD is gone; now on net 5V_APM: R5.2
- net 5V_APM: now also J3.1 (Pin_1)
- net DSM_I2C1_SCL: now also J3.3 (Pin_3)
- net DSM_I2C1_SDA: now also J3.2 (Pin_2)
- net GND: now also J3.4 (Pin_4)
Other:
- removed sheet DSM_debug
Changed lines of the file:
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@@
 		)
 	)
+	(junction
+		(at 146.05 102.87)
+		(diameter 0)
+		(color 0 0 0 0)
+	)
 	(no_connect
 		(at 143.51 107.95)
@@
 	(wire
 		(pts
+			(xy 146.05 100.33) (xy 146.05 102.87)
+		)
+		(stroke
+			(width 0)
+			(type default)
+		)
+	)
+	(wire
+		(pts
 			(xy 109.22 215.9) (xy 110.49 215.9)
 		)
@@
 	(wire
 		(pts
-			(xy 82.55 114.3) (xy 68.58 114.3)
+			(xy 146.05 102.87) (xy 143.51 102.87)
 		)
 		(stroke
@@
 	(wire
 		(pts
-			(xy 143.51 201.93) (xy 146.05 201.93)
+			(xy 146.05 102.87) (xy 148.59 102.87)
 		)
 		(stroke
@@
 	(wire
 		(pts
-			(xy 160.02 179.07) (xy 176.53 179.07)
+			(xy 143.51 201.93) (xy 146.05 201.93)
 		)
 		(stroke
@@
 	(wire
 		(pts
-			(xy 148.59 231.14) (xy 162.56 231.14)
+			(xy 160.02 179.07) (xy 176.53 179.07)
 		)
 		(stroke
@@
 	(wire
 		(pts
-			(xy 160.02 173.99) (xy 176.53 173.99)
+			(xy 148.59 231.14) (xy 162.56 231.14)
 		)
 		(stroke
@@
 	(wire
 		(pts
-			(xy 95.25 163.83) (xy 107.95 163.83)
+			(xy 160.02 173.99) (xy 176.53 173.99)
 		)
 		(stroke
@@
 	(wire
 		(pts
-			(xy 143.51 102.87) (xy 146.05 102.87)
-		)
-		(stroke
-			(width 0)
-			(type default)
-		)
-	)
-	(wire
-		(pts
-			(xy 82.55 118.11) (xy 68.58 118.11)
-		)
-		(stroke
-			(width 0)
-			(type default)
-		)
-	)
-	(wire
-		(pts
 			(xy 158.75 214.63) (xy 162.56 214.63)
 		)
@@
 	(wire
 		(pts
-			(xy 95.25 181.61) (xy 107.95 181.61)
-		)
-		(stroke
-			(width 0)
-			(type default)
-		)
-	)
-	(wire
-		(pts
 			(xy 162.56 128.27) (xy 176.53 128.27)
 		)
@@
 		)
 	)
-	(label "DSM_DBG_RX"
-		(at 82.55 114.3 180)
-		(effects
-			(font
-				(size 1.27 1.27)
-			)
-			(justify right bottom)
-		)
-	)
-	(label "DSM_DBG_TX"
-		(at 82.55 118.11 180)
-		(effects
-			(font
-				(size 1.27 1.27)
-			)
-			(justify right bottom)
-		)
-	)
 	(label "DSM_LED_FAIL"
 		(at 160.02 173.99 0)
@@
 		)
 	)
-	(label "DSM_DBG_RX"
-		(at 95.25 181.61 0)
-		(effects
-			(font
-				(size 1.27 1.27)
-			)
-			(justify left bottom)
-		)
-	)
 	(label "DSM_USB_D+"
 		(at 162.56 128.27 0)
@@
 		)
 	)
-	(label "DSM_DBG_TX"
-		(at 95.25 163.83 0)
-		(effects
-			(font
-				(size 1.27 1.27)
-			)
-			(justify left bottom)
-		)
-	)
 	(label "DSM_USB_D-"
 		(at 82.55 137.16 180)
@@
 		)
 	)
+	(hierarchical_label "DSM_DBG_TX"
+		(shape output)
+		(at 107.95 163.83 180)
+		(effects
+			(font
+				(size 1.27 1.27)
+			)
+			(justify right)
+		)
+	)
 	(hierarchical_label "DSM_FMC_NBL0"
 		(shape bidirectional)
@@
 		)
 	)
+	(hierarchical_label "DSM_DBG_RX"
+		(shape input)
+		(at 107.95 181.61 180)
+		(effects
+			(font
+				(size 1.27 1.27)
+			)
+			(justify right)
+		)
+	)
 	(hierarchical_label "DSM_FMC_D12"
 		(shape bidirectional)
@@
 		)
 	)
+	(hierarchical_label "DSM_VDD"
+		(shape output)
+		(at 148.59 102.87 0)
+		(effects
+			(font
+				(size 1.27 1.27)
+			)
+			(justify left)
+		)
+	)
 	(hierarchical_label "DSM_FMC_D9"
 		(shape bidirectional)
@@
 	)
 	(symbol
+		(lib_id "Connector_Generic:Conn_01x04")
+		(at 118.11 220.98 0)
+		(unit 1)
+		(exclude_from_sim no)
+		(in_bom yes)
+		(on_board yes)
+		(dnp no)
+		(fields_autoplaced yes)
+		(property "Reference" "J3"
+			(at 120.65 220.9799 0)
+			(effects
+				(font
+					(size 1.27 1.27)
+				)
+				(justify left)
+			)
+		)
+		(property "Value" "LCD_display"
+			(at 120.65 223.5199 0)
+			(effects
+				(font
+					(size 1.27 1.27)
+				)
+				(justify left)
+			)
+		)
+		(property "Footprint" "Connector_PinHeader_1.00mm:PinHeader_1x04_P1.00mm_Horizontal"
+			(at 118.11 220.98 0)
+			(effects
+				(font
+					(size 1.27 1.27)
+				)
+				(hide yes)
+			)
+		)
+		(property "Datasheet" "~"
+			(at 118.11 220.98 0)
+			(effects
+				(font
+					(size 1.27 1.27)
+				)
+				(hide yes)
+			)
+		)
+		(property "Description" "Generic connector, single row, 01x04, script generated (kicad-library-utils/schlib/autogen/connector/)"
+			(at 118.11 220.98 0)
+			(effects
+				(font
+					(size 1.27 1.27)
+				)
+				(hide yes)
+			)
+		)
+		(pin "3"
+		)
+		(pin "4"
+		)
+		(pin "2"
+		)
+		(pin "1"
+		)
+		(instances
+			(project "signalmesh"
+				(path "/fe7b15e9-f0ed-4338-9f03-dd7651dace13/4391c51f-6ab5-4b63-a6de-56382e56f1df"
+					(reference "J3")
+					(unit 1)
+				)
+			)
+		)
+	)
+	(symbol
 		(lib_id "Device:LED")
 		(at 203.2 218.44 270)
@@
 	(symbol
 		(lib_id "power:+5V")
-		(at 146.05 102.87 0)
+		(at 146.05 100.33 0)
 		(unit 1)
 		(exclude_from_sim no)
@@
 		(fields_autoplaced yes)
 		(property "Reference" "#PWR0102"
-			(at 146.05 106.68 0)
+			(at 146.05 104.14 0)
 			(effects
 				(font
@@
 		)
 		(property "Value" "5V_APM"
-			(at 148.59 101.5999 0)
+			(at 148.59 99.0599 0)
 			(effects
 				(font
@@
 		)
 		(property "Footprint" ""
-			(at 146.05 102.87 0)
+			(at 146.05 100.33 0)
 			(effects
 				(font
@@
 		)
 		(property "Datasheet" ""
-			(at 146.05 102.87 0)
+			(at 146.05 100.33 0)
 			(effects
 				(font
@@
 		)
 		(property "Description" "Power symbol creates a global label with name \"+5V\""
-			(at 146.05 102.87 0)
+			(at 146.05 100.33 0)
 			(effects
 				(font
@@
 	)
 	(symbol
-		(lib_id "Connector_Generic:Conn_01x04")
-		(at 118.11 220.98 0)
-		(unit 1)
-		(exclude_from_sim no)
-		(in_bom yes)
-		(on_board yes)
-		(dnp no)
-		(fields_autoplaced yes)
-		(property "Reference" "J17"
-			(at 120.65 220.9799 0)
-			(effects
-				(font
-					(size 1.27 1.27)
-				)
-				(justify left)
-			)
-		)
-		(property "Value" "LCD_display"
-			(at 120.65 223.5199 0)
-			(effects
-				(font
-					(size 1.27 1.27)
-				)
-				(justify left)
-			)
-		)
-		(property "Footprint" "Connector_PinHeader_1.00mm:PinHeader_1x04_P1.00mm_Vertical_SMD_Pin1Left"
-			(at 118.11 220.98 0)
-			(effects
-				(font
-					(size 1.27 1.27)
-				)
-				(hide yes)
-			)
-		)
-		(property "Datasheet" "~"
-			(at 118.11 220.98 0)
-			(effects
-				(font
-					(size 1.27 1.27)
-				)
-				(hide yes)
-			)
-		)
-		(property "Description" "Generic connector, single row, 01x04, script generated (kicad-library-utils/schlib/autogen/connector/)"
-			(at 118.11 220.98 0)
-			(effects
-				(font
-					(size 1.27 1.27)
-				)
-				(hide yes)
-			)
-		)
-		(pin "3"
-		)
-		(pin "4"
-		)
-		(pin "2"
-		)
-		(pin "1"
-		)
-		(instances
-			(project "signalmesh"
-				(path "/fe7b15e9-f0ed-4338-9f03-dd7651dace13/4391c51f-6ab5-4b63-a6de-56382e56f1df"
-					(reference "J17")
-					(unit 1)
-				)
-			)
-		)
-	)
-	(symbol
 		(lib_id "power:GND")
 		(at 199.39 214.63 0)
@@
 				)
 			)
-		)
-	)
-	(sheet
-		(at 53.34 110.49)
-		(size 15.24 11.43)
-		(exclude_from_sim no)
-		(in_bom yes)
-		(on_board yes)
-		(dnp no)
-		(fields_autoplaced yes)
-		(stroke
-			(width 0.1524)
-			(type solid)
-		)
-		(fill
-			(color 0 0 0 0.0000)
-		)
-		(property "Sheetname" "DSM_debug"
-			(at 53.34 109.7784 0)
-			(effects
-				(font
-					(size 1.27 1.27)
-				)
-				(justify left bottom)
-			)
-		)
-		(property "Sheetfile" "DSM_debug.kicad_sch"
-			(at 53.34 122.5046 0)
-			(effects
-				(font
-					(size 1.27 1.27)
-				)
-				(justify left top)
-			)
-		)
-		(pin "DSM_DBG_TX" input
-			(at 68.58 114.3 0)
-			(effects
-				(font
-					(size 1.27 1.27)
-				)
-				(justify right)
-			)
-		)
-		(pin "DSM_DBG_RX" input
-			(at 68.58 118.11 0)
-			(effects
-				(font
-					(size 1.27 1.27)
-				)
-				(justify right)
-			)
-		)
-		(instances
-			(project "signalmesh"
-				(path "/fe7b15e9-f0ed-4338-9f03-dd7651dace13/4391c51f-6ab5-4b63-a6de-56382e56f1df"
-					(page "10")
-				)
-			)
