File: schematic/v2/backupdebugs/ACM_debug.kicad_sch (KiCad schematic)
At the start: 16 parts, among them J13 UUM_DBG, J24 USB_A, U35 CH340G, Y4 Crystal

Commit message: time to start routing?
Parts:
- removed C20, C21, C22: 22pf, Capacitor_SMD:C_0805_2012Metric, symbol Device:C_Small
- removed D46, D47: LED_PWR, LED_SMD:LED_0603_1608Metric, symbol Device:LED
- removed D48: TXD, LED_SMD:LED_0603_1608Metric, symbol Device:LED
- removed D49: RXD, LED_SMD:LED_0603_1608Metric, symbol Device:LED
- removed J13: UUM_DBG, Connector_PinHeader_1.00mm:PinHeader_1x03_P1.00mm_Horizontal, symbol Connector_Generic:Conn_01x03
- removed J24: USB_A, Connector_USB:USB_A_CNCTech_1001-011-01101_Horizontal, symbol Connector:USB_A
- removed R67, R68, R69, R70: 300, Resistor_SMD:R_0805_2012Metric_Pad1.20x1.40mm_HandSolder, symbol Device:R
- removed R71: 1k5, Resistor_SMD:R_0805_2012Metric_Pad1.20x1.40mm_HandSolder, symbol Device:R
- removed U35: CH340G, Package_SO:SOIC-16_3.9x9.9mm_P1.27mm, symbol Interface_USB:CH340G
- removed Y4: Crystal, symbol Device:Crystal
- added C11, C12, C13: 22pf, Capacitor_SMD:C_0805_2012Metric, symbol Device:C_Small
- added D33, D34: LED_PWR, LED_SMD:LED_0603_1608Metric, symbol Device:LED
- added D35: TXD, LED_SMD:LED_0603_1608Metric, symbol Device:LED
- added D36: RXD, LED_SMD:LED_0603_1608Metric, symbol Device:LED
- added J12: USB_A, Connector_USB:USB_A_CNCTech_1001-011-01101_Horizontal, symbol Connector:USB_A
- added J14: ACM_DBG, Connector_PinHeader_1.00mm:PinHeader_1x03_P1.00mm_Horizontal, symbol Connector_Generic:Conn_01x03
- added R51, R52, R53, R54: 300, Resistor_SMD:R_0805_2012Metric_Pad1.20x1.40mm_HandSolder, symbol Device:R
- added R55: 1k5, Resistor_SMD:R_0805_2012Metric_Pad1.20x1.40mm_HandSolder, symbol Device:R
- added U32: CH340G, Package_SO:SOIC-16_3.9x9.9mm_P1.27mm, symbol Interface_USB:CH340G
- added Y6: 12MHz, Crystal:Crystal_C26-LF_D2.1mm_L6.5mm_Horizontal, symbol Device:Crystal
Connections:
- net GND: now also C11.1, C12.2, C13.2, D33.1 (K), D34.1 (K), D35.1 (K), D36.1 (K), J12.4 (GND), J14.3 (Pin_3), U32.1 (GND)
- new net: C12.1, U32.7 (XI), Y6.1
- new net: J12.2 (D-), U32.6 (UD-)
- new net: J12.3 (D+), U32.5 (UD+)
- new net: C13.1, U32.8 (XO), Y6.2
- new net: D36.2 (A), R54.2
- new net: D34.2 (A), R52.1
- new net: D35.2 (A), R53.2
- new net: D33.2 (A), R51.1
- new net ACM_DBG_RX: J14.2 (Pin_2), R53.1, R54.1, R55.1, U32.2 (TXD), U32.3 (RXD)
- new net ACM_DBG_TX: J14.1 (Pin_1), R55.2
- new net ACM_VDD: C11.2, J12.1 (VBUS), R51.2, R52.2, U32.16 (VCC)
Other:
- note added: "ACM Debug Port"
- note added: "ACM USB2.0 DBG PORT"
- note removed: "UUM Debug Port"
- note removed: "UUM USB2.0 DBG PORT"
